File: KiCad/Radio-86RK.kicad_sch (KiCad schematic)
At the start: 17 parts, among them SW68 Reset, U1 8080A/КР580ВМ80А, U12 74LS373/К555ИР22, U14 74LS138/К555ИД7, U16 7486/К155ЛП5, U17 7474/К155ТМ2, U18 7408/К155ЛИ1, U19 7404/К155ЛН1, U2 8224/КР580ГФ24, U20 7400/К155ЛА3, U27 DS1233, U7 8257/КР580ВТ57, Y1 16MHz

Commit message: Relink R1-R15 to official Resistor_THT footprint
The 15 discrete resistors used My_Components:Res_762, an unresolved
library nickname with no fp-lib-table entry anywhere on disk. Compared
the footprint against the actual ordered part (Stackpole CF14 1/4W
carbon film, per the README Mouser BOM) rather than just the closest
official name: the real part's datasheet body (6.50x2.30mm) is closer
to Resistor_THT:R_Axial_DIN0207_L6.3mm_D2.5mm_P7.62mm_Horizontal's
silkscreen outline (6.54x2.74mm) than to the project's own hand-drawn
one (5.84x2.03mm), so the official footprint is the more accurate
choice, not just a fallback. Same 7.62mm pin pitch, and it comes with
a working 3D model - the project's own model reference
("discret/resistor.wrl") doesn't resolve on any current KiCad install.

Co-Authored-By: Claude Sonnet 5 <noreply@anthropic.com>
Parts:
- R6: footprint My_Components:Res_762 -> Resistor_THT:R_Axial_DIN0207_L6.3mm_D2.5mm_P7.62mm_Horizontal
Changed lines of the file:
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@@
 			)
 		)
-		(property "Footprint" "My_Components:Res_762"
+		(property "Footprint" "Resistor_THT:R_Axial_DIN0207_L6.3mm_D2.5mm_P7.62mm_Horizontal"
 			(at 44.45 49.022 90)
 			(hide yes)

Commit message: Relink ceramic capacitors and F1 polyfuse to official footprints
The 39 refs (C1-C32, C39-C44, F1) used My_Components:Cap_Cer_508, an
unresolved library nickname. Resolved the real ordered parts from the
README Mouser BOM: C1-C32 are Vishay K104K15X7RF53H5 (~4.0x4.0x2.6mm
body), C40-C44 are TDK FG28-series (~4.0x5.5mm body), C39 is TDK
FG24-series (~4.5x5.5mm, larger), and F1 is a Littelfuse 16R110BU PTC
resettable fuse with no dedicated KiCad footprint.

All share the project's existing 5.08mm pitch (matches every
datasheet's 5.0mm +/-0.8-1.0mm spec). Split into two official
Capacitor_THT footprints matching the two real body-size groups
(C_Disc_D4.7mm_W2.5mm_P5.00mm for the smaller Vishay/FG28 parts,
C_Disc_D5.1mm_W3.2mm_P5.00mm for the larger FG24 C39) rather than
forcing one footprint on parts of two different real sizes. F1 reuses
the small-cap disc footprint since Littelfuse's radial PTC package at
this pitch is mechanically a disc shape with no official equivalent.

Co-Authored-By: Claude Sonnet 5 <noreply@anthropic.com>
Parts:
- C43, C44: footprint My_Components:Cap_Cer_508 -> Capacitor_THT:C_Disc_D4.7mm_W2.5mm_P5.00mm
Changed lines of the file:
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@@
 			)
 		)
-		(property "Footprint" "My_Components:Cap_Cer_508"
+		(property "Footprint" "Capacitor_THT:C_Disc_D4.7mm_W2.5mm_P5.00mm"
 			(at 31.4452 60.96 0)
 			(hide yes)
@@
 			)
 		)
-		(property "Footprint" "My_Components:Cap_Cer_508"
+		(property "Footprint" "Capacitor_THT:C_Disc_D4.7mm_W2.5mm_P5.00mm"
 			(at 38.1 36.5252 0)
 			(hide yes)

Commit message: Relink transistors Q1/Q2 and U27 to official TO-92 footprint
Q1/Q2 are 2N3904 (standard EBC pinout); U27 is a DS1233-5 CPU
supervisor, electrically unrelated but also a genuine 3-pin TO-92
package (GND/RESET/VCC). Verified both real pinouts already match the
existing pad-to-net mapping (pad1/2/3 = E/B/C for the 2N3904s,
GND/RESET/VCC for the DS1233) - footprint pad numbers are position
slots, not semantics, so this carries no pin-swap risk.

All three share identical 2.54mm inline pad spacing; official
Package_TO_SOT_THT:TO-92_Inline_Wide is an exact match ("TO-92 leads
in-line, wide", NXP SOT54/SC-43A - precisely this hand-formed
straight-lead mounting style).

Corrected the anchor-point placement shift (old footprint centered on
pad 2, official anchors at pad 1) immediately this time rather than
after the fact - verified via DRC that no track_dangling/starved_thermal
regressions appeared, unlike the first pass on R/C/D.

Co-Authored-By: Claude Sonnet 5 <noreply@anthropic.com>
Parts:
- U27: footprint My_Components:Transistor_TO92_EBC_254 -> Package_TO_SOT_THT:TO-92_Inline_Wide
Changed lines of the file:
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@@
 			)
 		)
-		(property "Footprint" "My_Components:Transistor_TO92_EBC_254"
+		(property "Footprint" "Package_TO_SOT_THT:TO-92_Inline_Wide"
 			(at 17.78 58.42 0)
 			(hide yes)
