File: KiCad/Radio-86RK.kicad_sch (KiCad schematic)
At the start: 17 parts, among them SW68 Reset, U1 8080A/КР580ВМ80А, U12 74LS373/К555ИР22, U14 74LS138/К555ИД7, U16 7486/К155ЛП5, U17 7474/К155ТМ2, U18 7408/К155ЛИ1, U19 7404/К155ЛН1, U2 8224/КР580ГФ24, U20 7400/К155ЛА3, U27 DS1233, U7 8257/КР580ВТ57, Y1 16MHz

Commit message: Relink Y1 (16MHz HC-49U crystal) to the official footprint
Real part is Abracon ATS160-E (Mouser 774-ATS160-E), a 16MHz
series-resonant HC-49U crystal. Relinked to the official
Crystal:Crystal_HC49-U_Vertical footprint, which includes a bundled
STEP 3D model. Pad pitch (4.88mm) matches the project's original
(4.88188mm) to within rounding; pad/drill size is a closer fit to
real HC-49U leads (1.5mm/0.8mm vs. the original's 1.397mm/0.8128mm).

Official footprint anchors at pad1 (local origin) versus the
project's center-anchored instance. Solved for the correction via
the established rotation transform (180° rotation unchanged,
position (16.411, 80.01) = old pad1 world location) and verified
both pads land within 0.002mm of their pre-swap world positions,
nets unchanged (Net-(C44-Pad2), Net-(U2-XTAL1)).

DRC lib_footprint_issues 29 -> 28.
Parts:
- Y1: footprint My_Components:Crystal_HC-49U_Vert -> Crystal:Crystal_HC49-U_Vertical
Changed lines of the file:
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@@
 			)
 		)
-		(property "Footprint" "My_Components:Crystal_HC-49U_Vert"
+		(property "Footprint" "Crystal:Crystal_HC49-U_Vertical"
 			(at 41.91 27.94 0)
 			(hide yes)

Commit message: Relink SW68 (B3F-3152 6mm tactile switch) to a materialized custom footprint
Real part is Omron B3F-3152 (Mouser 653-B3F-3152), a 6mm right-angle
tactile switch. The official KiCad candidate
(Button_Switch_THT:SW_SPST_Omron_B3F-315x_Angled) initially looked
like a match, but its two ground/mounting-leg pads sit on the
opposite side relative to the electrical pins compared to what the
board's existing copper requires - verified algebraically that no
single rotation could reconcile both the electrical pin pair and the
ground-pad pair simultaneously against the official footprint, only
a mirror would, which would imply a genuine chirality mismatch.

Sourced the manufacturer's own KiCad library export for this exact
part instead (SamacSys/Ultra Librarian) - its ground pads sit at the
opposite Y sign from the official KiCad footprint's, and with this
real geometry a plain 180° rotation reconciles all 4 pads exactly,
no mirror needed. This confirms the community-maintained official
footprint has an inaccuracy for this part, not the project's
original board layout. Ground/mounting pads renamed from the
manufacturer's numbered "3"/"4" to "GND" (duplicate pad name) to
match the project's schematic symbol pin. Includes the manufacturer's
real STEP 3D model.

New footprint anchors at pad1 (local origin); position (23.84298,
8.93064) = old pad1 world location, rotation 180°. Verified all 4
pads land within 0.001mm of their pre-swap world positions, nets
unchanged (Net-(U2-~{RESIN}), GND).

DRC lib_footprint_issues 25 -> 24.
Parts:
- SW68: footprint My_Components:Switch_Tactile_6mm_Right -> Switch_Tactile_Custom:B3F-3152
Changed lines of the file:
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@@
 			)
 		)
-		(property "Footprint" "My_Components:Switch_Tactile_6mm_Right"
+		(property "Footprint" "Switch_Tactile_Custom:B3F-3152"
 			(at 22.86 60.96 0)
 			(hide yes)
