File: KiCad/Radio-86RK.kicad_sch (KiCad schematic)
At the start: 17 parts, among them SW68 Reset, U1 8080A/КР580ВМ80А, U12 74LS373/К555ИР22, U14 74LS138/К555ИД7, U16 7486/К155ЛП5, U17 7474/К155ТМ2, U18 7408/К155ЛИ1, U19 7404/К155ЛН1, U2 8224/КР580ГФ24, U20 7400/К155ЛА3, U27 DS1233, U7 8257/КР580ВТ57, Y1 16MHz

Commit message: Relink U15-U20 (14-pin DIP 74LS-series logic) to the socket+chip composite footprint
Package width confirmed 300mil DIP-14 for the 74LS family (SN74LS00N: TI "N
package" PDIP-14), matching the board's existing 7.62mm row spacing. Reuses
the Task 23 IC_Socket_Custom compositing approach: pads/silkscreen from the
official Package_DIP:DIP-14_W7.62mm_Socket footprint, plus two composited
3D models (official socket STEP at board level, official chip STEP raised
5.48mm - real stack height of the BOM socket, Mouser 649-DILB14P-223TLF).

All 6 references are multi-unit symbols with redundant per-unit Footprint
property copies spread across up to 4 sheet files each (26 unit-instance
copies total) - batch_edit_schematic_components only patches one instance
per reference per call, so remaining stragglers were located and verified
by reference before a direct text substitution.

Anchor point moved from array-center to pad1 and rotation recomputed
180 (from F8's preserved 90) per instance, verified: all six show the
correct universal 74-series DIP-14 power pinout (pad7=GND, pad14=VCC),
and U15's full pad/net list matches the pre-swap board exactly.

Co-Authored-By: Claude Sonnet 5 <noreply@anthropic.com>
Parts:
- U16, U17, U18, U19, U20: footprint My_Components:IC_DIP14_300 -> IC_Socket_Custom:DIP-14_W7.62mm_Socketed
Changed lines of the file:
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@@
 			)
 		)
-		(property "Footprint" "My_Components:IC_DIP14_300"
+		(property "Footprint" "IC_Socket_Custom:DIP-14_W7.62mm_Socketed"
 			(at 91.44 154.94 0)
 			(hide yes)
@@
 			)
 		)
-		(property "Footprint" "My_Components:IC_DIP14_300"
+		(property "Footprint" "IC_Socket_Custom:DIP-14_W7.62mm_Socketed"
 			(at 124.46 175.26 0)
 			(hide yes)
@@
 			)
 		)
-		(property "Footprint" "My_Components:IC_DIP14_300"
+		(property "Footprint" "IC_Socket_Custom:DIP-14_W7.62mm_Socketed"
 			(at 124.46 190.5 0)
 			(hide yes)
@@
 			)
 		)
-		(property "Footprint" "My_Components:IC_DIP14_300"
+		(property "Footprint" "IC_Socket_Custom:DIP-14_W7.62mm_Socketed"
 			(at 203.2 81.28 0)
 			(hide yes)
@@
 			)
 		)
-		(property "Footprint" "My_Components:IC_DIP14_300"
+		(property "Footprint" "IC_Socket_Custom:DIP-14_W7.62mm_Socketed"
 			(at 233.68 53.34 0)
 			(hide yes)
@@
 			)
 		)
-		(property "Footprint" "My_Components:IC_DIP14_300"
+		(property "Footprint" "IC_Socket_Custom:DIP-14_W7.62mm_Socketed"
 			(at 213.36 50.8 0)
 			(hide yes)
@@
 			)
 		)
-		(property "Footprint" "My_Components:IC_DIP14_300"
+		(property "Footprint" "IC_Socket_Custom:DIP-14_W7.62mm_Socketed"
 			(at 182.88 88.9 0)
 			(hide yes)
@@
 			)
 		)
-		(property "Footprint" "My_Components:IC_DIP14_300"
+		(property "Footprint" "IC_Socket_Custom:DIP-14_W7.62mm_Socketed"
 			(at 213.36 63.5 0)
 			(hide yes)
@@
 			)
 		)
-		(property "Footprint" "My_Components:IC_DIP14_300"
+		(property "Footprint" "IC_Socket_Custom:DIP-14_W7.62mm_Socketed"
 			(at 182.88 71.12 0)
 			(hide yes)
@@
 			)
 		)
-		(property "Footprint" "My_Components:IC_DIP14_300"
+		(property "Footprint" "IC_Socket_Custom:DIP-14_W7.62mm_Socketed"
 			(at 233.68 66.04 0)
 			(hide yes)

Commit message: Relink U2/U14/U22 (16-pin DIP ICs) to the socket+chip composite footprint
Package width confirmed 300mil DIP-16 against the Intel 8224 datasheet
("16-Lead Cerdip Package") and TI SN75154N datasheet ("N PDIP 16", 13.97mm
tube width - the same standard TI 300mil tube spec confirmed for SN75150P
in Task 23); 74LS138 already covered by the Task 24 74LS-family confirmation.
Matches the board's existing 7.62mm row spacing.

Reuses the Task 23 IC_Socket_Custom compositing approach: pads/silkscreen
from the official Package_DIP:DIP-16_W7.62mm_Socket footprint, plus two
composited 3D models (official socket STEP at board level, official chip
STEP raised 5.48mm - real stack height of the BOM socket, Mouser
649-DILB16P-223TLF, per Arrow/Mouser structured spec data).

All three are single-unit symbols with one placement each - no multi-unit
stragglers this time. Anchor point moved from array-center to pad1 and
rotation recomputed 180 (from F8's preserved 90) per instance; U2's full
pad/net list matches the pre-swap board exactly, and U14/U22 both show
correct standard pinouts (74LS138 pin8=GND/pin16=VCC; SN75154N pin8=GND).

Co-Authored-By: Claude Sonnet 5 <noreply@anthropic.com>
Parts:
- U14, U2: footprint My_Components:IC_DIP16_300 -> IC_Socket_Custom:DIP-16_W7.62mm_Socketed
Changed lines of the file:
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@@
 			)
 		)
-		(property "Footprint" "My_Components:IC_DIP16_300"
+		(property "Footprint" "IC_Socket_Custom:DIP-16_W7.62mm_Socketed"
 			(at 66.04 43.18 0)
 			(hide yes)
@@
 			)
 		)
-		(property "Footprint" "My_Components:IC_DIP16_300"
+		(property "Footprint" "IC_Socket_Custom:DIP-16_W7.62mm_Socketed"
 			(at 185.42 35.56 0)
 			(hide yes)

Commit message: Relink U12 (74LS373 20-pin DIP) to the socket+chip composite footprint
Package width confirmed 300mil DIP-20 for SN74LS373N (TI: "20-PDIP"), matching
the board's existing 7.62mm row spacing - notable because 20-pin DIPs aren't
safely assumed from the 74LS-family pattern alone (some 20-pin parts use
600mil), so this one was checked explicitly per the plan.

Reuses the Task 23 IC_Socket_Custom compositing approach: pads/silkscreen
from the official Package_DIP:DIP-20_W7.62mm_Socket footprint, plus two
composited 3D models (official socket STEP at board level, official chip
STEP raised 5.48mm). Unlike Tasks 24/25, no source gave an explicit stack
height for this exact socket P/N (Mouser 649-DILB20P-223TLF); 5.48mm is
carried over from the same Amphenol TLF-family height confirmed directly
for the 14-pin and 16-pin sockets - flagged as an inference in the
footprint's descr field, and confirmed with the user before proceeding.

Anchor point moved from array-center to pad1 and rotation recomputed 180
(from F8's preserved 90); full pad/net list matches the pre-swap board
exactly.

Co-Authored-By: Claude Sonnet 5 <noreply@anthropic.com>
Parts:
- U12: footprint My_Components:IC_DIP20_300 -> IC_Socket_Custom:DIP-20_W7.62mm_Socketed
Changed lines of the file:
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@@
 			)
 		)
-		(property "Footprint" "My_Components:IC_DIP20_300"
+		(property "Footprint" "IC_Socket_Custom:DIP-20_W7.62mm_Socketed"
 			(at 129.54 142.24 0)
 			(hide yes)
