File: KiCad/Radio-86RK.kicad_sch (KiCad schematic)
At the start: 17 parts, among them SW68 Reset, U1 8080A/КР580ВМ80А, U12 74LS373/К555ИР22, U14 74LS138/К555ИД7, U16 7486/К155ЛП5, U17 7474/К155ТМ2, U18 7408/К155ЛИ1, U19 7404/К155ЛН1, U2 8224/КР580ГФ24, U20 7400/К155ЛА3, U27 DS1233, U7 8257/КР580ВТ57, Y1 16MHz

Commit message: Relink U1/U5/U6/U7/U8 (40-pin DIP ICs) to the socket+chip composite footprint
Package width confirmed 600mil DIP-40 - the board's own measured 15.24mm row
spacing already matched Package_DIP:DIP-40_W15.24mm exactly, and the Intel
8080A/8255A/8257/8275 family is universally packaged in standard 40-pin
plastic DIP with no narrow-body variant.

Reuses the Task 23 IC_Socket_Custom compositing approach: pads/silkscreen
from the official Package_DIP:DIP-40_W15.24mm_Socket footprint, plus two
composited 3D models (official socket STEP at board level, official chip
STEP raised 5.48mm - stack height directly confirmed for the BOM socket,
Mouser 649-DILB40P223TLF).

Anchor point moved from array-center to pad1 and rotation recomputed 180
(from F8's preserved 90) per instance; U1's full pad/net list matches the
pre-swap board exactly, and U5/U6/U7/U8 all show correct standard 40-pin
pinouts (GND/VCC at the expected positions).

This is the last unresolved My_Components reference in the project - DRC
confirms the "lib_footprint_issues" category has dropped to 0 (from 21
after Task 23), matching the plan's expected end state for the IC tasks.

Co-Authored-By: Claude Sonnet 5 <noreply@anthropic.com>
Parts:
- U1, U7: footprint My_Components:IC_DIP40_600 -> IC_Socket_Custom:DIP-40_W15.24mm_Socketed
Changed lines of the file:
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@@
 			)
 		)
-		(property "Footprint" "My_Components:IC_DIP40_600"
+		(property "Footprint" "IC_Socket_Custom:DIP-40_W15.24mm_Socketed"
 			(at 132.08 58.42 0)
 			(hide yes)
@@
 			)
 		)
-		(property "Footprint" "My_Components:IC_DIP40_600"
+		(property "Footprint" "IC_Socket_Custom:DIP-40_W15.24mm_Socketed"
 			(at 63.5 149.86 0)
 			(hide yes)
