File: KiCad/Radio-86RK.kicad_sch (KiCad schematic)
At the start: 17 parts, among them SW68 Reset, U1 8080A/КР580ВМ80А, U12 74LS373/К555ИР22, U14 74LS138/К555ИД7, U16 7486/К155ЛП5, U17 7474/К155ТМ2, U18 7408/К155ЛИ1, U19 7404/К155ЛН1, U2 8224/КР580ГФ24, U20 7400/К155ЛА3, U27 DS1233, U7 8257/КР580ВТ57, Y1 16MHz

Commit message: Re-home DS1233 (reset supervisor) from lost my_components library
Step 3/18. Relinks U27 on the root sheet from my_components:DS1233 to
Radio86RK_Custom:DS1233.
Parts:
- U27: symbol my_components:DS1233 -> Radio86RK_Custom:DS1233
Changed lines of the file:
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@@
 	)
 	(symbol
-		(lib_id "my_components:DS1233")
+		(lib_id "Radio86RK_Custom:DS1233")
 		(at 17.78 43.18 0)
 		(unit 1)

Commit message: Re-home 8080A (CPU) from lost my_components library
Step 4/18. Relinks U1 on the root sheet from my_components:8080A to
Radio86RK_Custom:8080A.
Parts:
- U1: symbol my_components:8080A -> Radio86RK_Custom:8080A
Changed lines of the file:
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@@
 	)
 	(symbol
-		(lib_id "my_components:8080A")
+		(lib_id "Radio86RK_Custom:8080A")
 		(at 132.08 58.42 0)
 		(unit 1)

Commit message: Re-home 8224 (clock generator/driver) from lost my_components library
Step 5/18. Relinks U2 on the root sheet from my_components:8224 to
Radio86RK_Custom:8224.
Parts:
- U2: symbol my_components:8224 -> Radio86RK_Custom:8224
Changed lines of the file:
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@@
 	)
 	(symbol
-		(lib_id "my_components:8224")
+		(lib_id "Radio86RK_Custom:8224")
 		(at 66.04 41.91 0)
 		(unit 1)

Commit message: Re-home 8257 (DMA controller) from lost my_components library
Step 6/18. Relinks U7 on the root sheet from my_components:8257 to
Radio86RK_Custom:8257.
Parts:
- U7: symbol my_components:8257 -> Radio86RK_Custom:8257
Changed lines of the file:
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@@
 	)
 	(symbol
-		(lib_id "my_components:8257")
+		(lib_id "Radio86RK_Custom:8257")
 		(at 63.5 144.78 0)
 		(unit 1)

Commit message: Re-home Switch_Tactile_Vertical (reset button) from lost my_components library
Step 17/18. Relinks SW68 on the root sheet from
my_components:Switch_Tactile_Vertical to
Radio86RK_Custom:Switch_Tactile_Vertical.

Unlike the original monolithic relink commit (28c05ca on migrate2kicad10),
this text-level lib_id swap never touches the instance's (at ...)/(mirror
x) placement transform, so SW68's mirror is preserved automatically --
no separate mirror-restore edit needed here.
Parts:
- SW68: symbol my_components:Switch_Tactile_Vertical -> Radio86RK_Custom:Switch_Tactile_Vertical
Changed lines of the file:
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@@
 	)
 	(symbol
-		(lib_id "my_components:Switch_Tactile_Vertical")
+		(lib_id "Radio86RK_Custom:Switch_Tactile_Vertical")
 		(at 22.86 60.96 90)
 		(mirror x)
