File: KiCad/Radio-86RK-Power.kicad_sch (KiCad schematic)
At the start: 52 parts, among them J2 5V, J3 Power, J7 Extension, U16 7486/К155ЛП5, U17 7474/К155ТМ2, U18 7408/К155ЛИ1, U19 7404/К155ЛН1, U20 7400/К155ЛА3, U25 LM7905/КР1179ЕН5В, U26 IZ0512S

Commit message: Relink ceramic capacitors and F1 polyfuse to official footprints
The 39 refs (C1-C32, C39-C44, F1) used My_Components:Cap_Cer_508, an
unresolved library nickname. Resolved the real ordered parts from the
README Mouser BOM: C1-C32 are Vishay K104K15X7RF53H5 (~4.0x4.0x2.6mm
body), C40-C44 are TDK FG28-series (~4.0x5.5mm body), C39 is TDK
FG24-series (~4.5x5.5mm, larger), and F1 is a Littelfuse 16R110BU PTC
resettable fuse with no dedicated KiCad footprint.

All share the project's existing 5.08mm pitch (matches every
datasheet's 5.0mm +/-0.8-1.0mm spec). Split into two official
Capacitor_THT footprints matching the two real body-size groups
(C_Disc_D4.7mm_W2.5mm_P5.00mm for the smaller Vishay/FG28 parts,
C_Disc_D5.1mm_W3.2mm_P5.00mm for the larger FG24 C39) rather than
forcing one footprint on parts of two different real sizes. F1 reuses
the small-cap disc footprint since Littelfuse's radial PTC package at
this pitch is mechanically a disc shape with no official equivalent.

Co-Authored-By: Claude Sonnet 5 <noreply@anthropic.com>
Parts:
- C1, C10, C11, C12, C13, C14, C15, C16, C17, C18, C19, C2, C20, C21, C22, C23, C24, C25, C26, C27, C28, C29, C3, C30, C4, C5, C6, C7, C8, C9: footprint My_Components:Cap_Cer_508 -> Capacitor_THT:C_Disc_D4.7mm_W2.5mm_P5.00mm
Changed lines of the file:
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@@
 			)
 		)
-		(property "Footprint" "My_Components:Cap_Cer_508"
+		(property "Footprint" "Capacitor_THT:C_Disc_D4.7mm_W2.5mm_P5.00mm"
 			(at 122.8852 43.18 0)
 			(hide yes)
@@
 			)
 		)
-		(property "Footprint" "My_Components:Cap_Cer_508"
+		(property "Footprint" "Capacitor_THT:C_Disc_D4.7mm_W2.5mm_P5.00mm"
 			(at 130.5052 43.18 0)
 			(hide yes)
@@
 			)
 		)
-		(property "Footprint" "My_Components:Cap_Cer_508"
+		(property "Footprint" "Capacitor_THT:C_Disc_D4.7mm_W2.5mm_P5.00mm"
 			(at 138.1252 43.18 0)
 			(hide yes)
@@
 			)
 		)
-		(property "Footprint" "My_Components:Cap_Cer_508"
+		(property "Footprint" "Capacitor_THT:C_Disc_D4.7mm_W2.5mm_P5.00mm"
 			(at 145.7452 43.18 0)
 			(hide yes)
@@
 			)
 		)
-		(property "Footprint" "My_Components:Cap_Cer_508"
+		(property "Footprint" "Capacitor_THT:C_Disc_D4.7mm_W2.5mm_P5.00mm"
 			(at 153.3652 43.18 0)
 			(hide yes)
@@
 			)
 		)
-		(property "Footprint" "My_Components:Cap_Cer_508"
+		(property "Footprint" "Capacitor_THT:C_Disc_D4.7mm_W2.5mm_P5.00mm"
 			(at 160.9852 43.18 0)
 			(hide yes)
@@
 			)
 		)
-		(property "Footprint" "My_Components:Cap_Cer_508"
+		(property "Footprint" "Capacitor_THT:C_Disc_D4.7mm_W2.5mm_P5.00mm"
 			(at 168.6052 43.18 0)
 			(hide yes)
@@
 			)
 		)
-		(property "Footprint" "My_Components:Cap_Cer_508"
+		(property "Footprint" "Capacitor_THT:C_Disc_D4.7mm_W2.5mm_P5.00mm"
 			(at 176.2252 43.18 0)
 			(hide yes)
@@
 			)
 		)
-		(property "Footprint" "My_Components:Cap_Cer_508"
+		(property "Footprint" "Capacitor_THT:C_Disc_D4.7mm_W2.5mm_P5.00mm"
 			(at 183.8452 43.18 0)
 			(hide yes)
@@
 			)
 		)
-		(property "Footprint" "My_Components:Cap_Cer_508"
+		(property "Footprint" "Capacitor_THT:C_Disc_D4.7mm_W2.5mm_P5.00mm"
 			(at 199.0852 43.18 0)
 			(hide yes)
@@
 			)
 		)
-		(property "Footprint" "My_Components:Cap_Cer_508"
+		(property "Footprint" "Capacitor_THT:C_Disc_D4.7mm_W2.5mm_P5.00mm"
 			(at 115.2652 58.42 0)
 			(hide yes)
@@
 			)
 		)
-		(property "Footprint" "My_Components:Cap_Cer_508"
+		(property "Footprint" "Capacitor_THT:C_Disc_D4.7mm_W2.5mm_P5.00mm"
 			(at 122.8852 58.42 0)
 			(hide yes)
@@
 			)
 		)
-		(property "Footprint" "My_Components:Cap_Cer_508"
+		(property "Footprint" "Capacitor_THT:C_Disc_D4.7mm_W2.5mm_P5.00mm"
 			(at 130.5052 58.42 0)
 			(hide yes)
@@
 			)
 		)
-		(property "Footprint" "My_Components:Cap_Cer_508"
+		(property "Footprint" "Capacitor_THT:C_Disc_D4.7mm_W2.5mm_P5.00mm"
 			(at 138.1252 58.42 0)
 			(hide yes)
@@
 			)
 		)
-		(property "Footprint" "My_Components:Cap_Cer_508"
+		(property "Footprint" "Capacitor_THT:C_Disc_D4.7mm_W2.5mm_P5.00mm"
 			(at 145.7452 58.42 0)
 			(hide yes)
@@
 			)
 		)
-		(property "Footprint" "My_Components:Cap_Cer_508"
+		(property "Footprint" "Capacitor_THT:C_Disc_D4.7mm_W2.5mm_P5.00mm"
 			(at 153.3652 58.42 0)
 			(hide yes)
@@
 			)
 		)
-		(property "Footprint" "My_Components:Cap_Cer_508"
+		(property "Footprint" "Capacitor_THT:C_Disc_D4.7mm_W2.5mm_P5.00mm"
 			(at 160.9852 58.42 0)
 			(hide yes)
@@
 			)
 		)
-		(property "Footprint" "My_Components:Cap_Cer_508"
+		(property "Footprint" "Capacitor_THT:C_Disc_D4.7mm_W2.5mm_P5.00mm"
 			(at 168.6052 58.42 0)
 			(hide yes)
@@
 			)
 		)
-		(property "Footprint" "My_Components:Cap_Cer_508"
+		(property "Footprint" "Capacitor_THT:C_Disc_D4.7mm_W2.5mm_P5.00mm"
 			(at 191.4652 43.18 0)
 			(hide yes)
@@
 			)
 		)
-		(property "Footprint" "My_Components:Cap_Cer_508"
+		(property "Footprint" "Capacitor_THT:C_Disc_D4.7mm_W2.5mm_P5.00mm"
 			(at 122.8852 91.44 0)
 			(hide yes)
@@
 			)
 		)
-		(property "Footprint" "My_Components:Cap_Cer_508"
+		(property "Footprint" "Capacitor_THT:C_Disc_D4.7mm_W2.5mm_P5.00mm"
 			(at 168.6052 104.14 0)
 			(hide yes)
@@
 			)
 		)
-		(property "Footprint" "My_Components:Cap_Cer_508"
+		(property "Footprint" "Capacitor_THT:C_Disc_D4.7mm_W2.5mm_P5.00mm"
 			(at 176.2252 104.14 0)
 			(hide yes)
@@
 			)
 		)
-		(property "Footprint" "My_Components:Cap_Cer_508"
+		(property "Footprint" "Capacitor_THT:C_Disc_D4.7mm_W2.5mm_P5.00mm"
 			(at 122.8852 104.14 0)
 			(hide yes)
@@
 			)
 		)
-		(property "Footprint" "My_Components:Cap_Cer_508"
+		(property "Footprint" "Capacitor_THT:C_Disc_D4.7mm_W2.5mm_P5.00mm"
 			(at 130.5052 91.44 0)
 			(hide yes)
@@
 			)
 		)
-		(property "Footprint" "My_Components:Cap_Cer_508"
+		(property "Footprint" "Capacitor_THT:C_Disc_D4.7mm_W2.5mm_P5.00mm"
 			(at 138.1252 91.44 0)
 			(hide yes)
@@
 			)
 		)
-		(property "Footprint" "My_Components:Cap_Cer_508"
+		(property "Footprint" "Capacitor_THT:C_Disc_D4.7mm_W2.5mm_P5.00mm"
 			(at 191.4652 58.42 0)
 			(hide yes)
@@
 			)
 		)
-		(property "Footprint" "My_Components:Cap_Cer_508"
+		(property "Footprint" "Capacitor_THT:C_Disc_D4.7mm_W2.5mm_P5.00mm"
 			(at 176.2252 58.42 0)
 			(hide yes)
@@
 			)
 		)
-		(property "Footprint" "My_Components:Cap_Cer_508"
+		(property "Footprint" "Capacitor_THT:C_Disc_D4.7mm_W2.5mm_P5.00mm"
 			(at 183.8452 58.42 0)
 			(hide yes)
@@
 			)
 		)
-		(property "Footprint" "My_Components:Cap_Cer_508"
+		(property "Footprint" "Capacitor_THT:C_Disc_D4.7mm_W2.5mm_P5.00mm"
 			(at 130.5052 104.14 0)
 			(hide yes)
@@
 			)
 		)
-		(property "Footprint" "My_Components:Cap_Cer_508"
+		(property "Footprint" "Capacitor_THT:C_Disc_D4.7mm_W2.5mm_P5.00mm"
 			(at 145.7452 91.44 0)
 			(hide yes)

Commit message: Relink electrolytic capacitors C33-C38 to official footprint
The real ordered part is KEMET A750EK476M1E (47uF/25V Radial Solid
Polymer Aluminum, case code EK: D6.3mm x L8mm, 2.5mm lead spacing) -
the project's existing pitch and footprint name already matched this
part exactly, so this is a clean swap: Capacitor_THT:CP_Radial_D6.3mm_P2.50mm
is an essentially exact match (same pitch, near-identical pad/drill,
same pad-numbering/polarity convention) and adds a working 3D model.

Co-Authored-By: Claude Sonnet 5 <noreply@anthropic.com>
Parts:
- C33, C34, C35, C36, C37: footprint My_Components:Cap_Elec_Radial_6.3mm -> Capacitor_THT:CP_Radial_D6.3mm_P2.50mm
Changed lines of the file:
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@@
 			)
 		)
-		(property "Footprint" "My_Components:Cap_Elec_Radial_6.3mm"
+		(property "Footprint" "Capacitor_THT:CP_Radial_D6.3mm_P2.50mm"
 			(at 205.74 54.61 0)
 			(hide yes)
@@
 			)
 		)
-		(property "Footprint" "My_Components:Cap_Elec_Radial_6.3mm"
+		(property "Footprint" "Capacitor_THT:CP_Radial_D6.3mm_P2.50mm"
 			(at 198.12 54.61 0)
 			(hide yes)
@@
 			)
 		)
-		(property "Footprint" "My_Components:Cap_Elec_Radial_6.3mm"
+		(property "Footprint" "Capacitor_THT:CP_Radial_D6.3mm_P2.50mm"
 			(at 152.4 87.63 0)
 			(hide yes)
@@
 			)
 		)
-		(property "Footprint" "My_Components:Cap_Elec_Radial_6.3mm"
+		(property "Footprint" "Capacitor_THT:CP_Radial_D6.3mm_P2.50mm"
 			(at 182.88 100.33 0)
 			(hide yes)
@@
 			)
 		)
-		(property "Footprint" "My_Components:Cap_Elec_Radial_6.3mm"
+		(property "Footprint" "Capacitor_THT:CP_Radial_D6.3mm_P2.50mm"
 			(at 137.16 100.33 0)
 			(hide yes)

Commit message: Relink mounting holes HOLE1-7 to a materialized custom footprint
HOLE1-7 are grounded M3 mounting holes (plated pad tied to GND, drill
3.048mm / pad 4.064mm) - not plain mechanical clearance holes. No
official KiCad MountingHole variant matches this: every net-connected
("Pad") variant at a ~3mm drill is fixed at 6mm pad OD by the
footprint generator (47% larger), and that's true across all Pad/
Pad_TopBottom/Pad_TopOnly variants checked. Forcing that would be a
real copper change on 7 already-placed holes for no benefit.

Same approach as Cherry_MX_Custom (commit daacbd7): materialized the
project's exact existing geometry into a new project-local
MountingHole_Custom.pretty library rather than accepting a
larger-than-necessary official substitute. No PCB change - pad,
drill, and position are identical before and after.

Also found and corrected a reference-to-sheet mapping error from
earlier in the task: HOLE1-7 are actually on the Power sheet, not
Keyboard as initially assumed from misreading parallel tool call
results (same mistake as the earlier U27 mixup).

Co-Authored-By: Claude Sonnet 5 <noreply@anthropic.com>
Parts:
- HOLE1, HOLE2, HOLE3, HOLE4, HOLE5, HOLE6, HOLE7: footprint My_Components:Hole_3mm -> MountingHole_Custom:Hole_3mm
Changed lines of the file:
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@@
 			)
 		)
-		(property "Footprint" "My_Components:Hole_3mm"
+		(property "Footprint" "MountingHole_Custom:Hole_3mm"
 			(at 262.89 76.2 0)
 			(hide yes)
@@
 			)
 		)
-		(property "Footprint" "My_Components:Hole_3mm"
+		(property "Footprint" "MountingHole_Custom:Hole_3mm"
 			(at 262.89 81.28 0)
 			(hide yes)
@@
 			)
 		)
-		(property "Footprint" "My_Components:Hole_3mm"
+		(property "Footprint" "MountingHole_Custom:Hole_3mm"
 			(at 262.89 86.36 0)
 			(hide yes)
@@
 			)
 		)
-		(property "Footprint" "My_Components:Hole_3mm"
+		(property "Footprint" "MountingHole_Custom:Hole_3mm"
 			(at 262.89 91.44 0)
 			(hide yes)
@@
 			)
 		)
-		(property "Footprint" "My_Components:Hole_3mm"
+		(property "Footprint" "MountingHole_Custom:Hole_3mm"
 			(at 262.89 96.52 0)
 			(hide yes)
@@
 			)
 		)
-		(property "Footprint" "My_Components:Hole_3mm"
+		(property "Footprint" "MountingHole_Custom:Hole_3mm"
 			(at 262.89 101.6 0)
 			(hide yes)
@@
 			)
 		)
-		(property "Footprint" "My_Components:Hole_3mm"
+		(property "Footprint" "MountingHole_Custom:Hole_3mm"
 			(at 262.89 106.68 0)
 			(hide yes)

Commit message: Relink J2 (2mm DC power jack) to a materialized custom footprint
My_Components:Conn_Power_Jack_Circular_Pads had no official KiCad
match: the only installed BarrelJack footprint for this Kycon family
(BarrelJack_Kycon_KLDX-0202-xC_Horizontal) is for the crimped-lead
"-xC" sibling part, not the straight-lead KLDX-0202-A actually used
here (Mouser 806-KLDX-0202-A). Pad spacing between the official
footprint and the project's own geometry matched almost exactly,
confirming the shell/hole pattern is shared across the family - only
lead style differs.

Sourced the manufacturer's own KiCad export (SamacSys/Ultra
Librarian) for the exact "-A" part, converted its legacy-format
footprint to modern KiCad 10 syntax, and registered it as
Conn_DCJack_Custom:KLDX-0202-A (round pads at pad1=(0,0) VCC/tip,
pad2=(-6.2,0) GND, pad3=(-3.2,4.7) GND - independently matching the
official crimped-variant footprint's pad2/pad3 coordinates), with the
manufacturer's STEP 3D model.

Corrected the anchor-point offset after forward-annotation: this
footprint anchors at pad 1, while the project's original anchored at
pad 2, so the placed position needed shifting by the pad1-pad2 vector
(same class of fix applied to every other relinked component this
migration). Rotation and net mapping (pad1=VCC, pad2/3=GND) were
unaffected. 3D model orientation verified visually.

Co-Authored-By: Claude Sonnet 5 <noreply@anthropic.com>
Parts:
- J2: footprint My_Components:Conn_Power_Jack_Circular_Pads -> Conn_DCJack_Custom:KLDX-0202-A
Changed lines of the file:
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@@
 			)
 		)
-		(property "Footprint" "My_Components:Conn_Power_Jack_Circular_Pads"
+		(property "Footprint" "Conn_DCJack_Custom:KLDX-0202-A"
 			(at 29.21 110.236 0)
 			(hide yes)

Commit message: Relink J3 (8-pin friction-lock header) to a materialized custom footprint
My_Components:Conn_Friction_Lock_8P_2.54mm had no official KiCad
match: the closest official candidate (generic
Connector_PinHeader_2.54mm:PinHeader_1x08_P2.54mm_Vertical) uses
slightly larger pads and, notably, arranges its 8 pins along local Y
rather than the local X this board's layout uses - the same
axis-arrangement gotcha already documented from the JP1/JP2 task.

Instead sourced the manufacturer's own KiCad export (SamacSys/Ultra
Librarian) for the exact real part (TE Connectivity/AMP 640456-8,
MTA-100 series, Mouser 571-6404568), registered as
Conn_FrictionLock_Custom:640456-8. This part-specific footprint
arranges its 8 pads along local X already (matching the board's
layout), uses pad sizing closer to the project's original
(1.725mm/1.15mm drill vs. the project's 1.524mm/1.016mm, vs. the
generic official candidate's 1.7mm/1.0mm), models the real shrouded
housing outline, and includes the manufacturer's STEP 3D model.

Corrected the anchor-point/rotation after forward-annotation: the
project's original footprint anchored at the body center (midpoint
of pins 4/5), while this footprint anchors at pad 1 with pad numbering
running in the opposite direction along X - requiring a position
shift to pad 1's original world coordinates plus a 180 degree
rotation. All 8 pads now land exactly on their pre-swap world
positions with unchanged net assignments (pad1-3=GND, pad4-6=VCC,
pad7=-12V, pad8=+12V). 3D model orientation verified visually.

Co-Authored-By: Claude Sonnet 5 <noreply@anthropic.com>
Parts:
- J3: footprint My_Components:Conn_Friction_Lock_8P_2.54mm -> Conn_FrictionLock_Custom:640456-8
Changed lines of the file:
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@@
 			)
 		)
-		(property "Footprint" "My_Components:Conn_Friction_Lock_8P_2.54mm"
+		(property "Footprint" "Conn_FrictionLock_Custom:640456-8"
 			(at 55.88 104.14 0)
 			(hide yes)
