File: KiCad/Radio-86RK-Power.kicad_sch (KiCad schematic)
At the start: 52 parts, among them J2 5V, J3 Power, J7 Extension, U16 7486/К155ЛП5, U17 7474/К155ТМ2, U18 7408/К155ЛИ1, U19 7404/К155ЛН1, U20 7400/К155ЛА3, U25 LM7905/КР1179ЕН5В, U26 IZ0512S

Commit message: Relink J7 (20x1 pin socket) to the official footprint
Real part is 3M/3M-ESD 929850-01-20-RB (Mouser 517-929850-01-20-RB),
a 20-position, 2.54mm-pitch, single-row through-hole female socket
strip. Relinked to the official Connector_PinSocket_2.54mm:
PinSocket_1x20_P2.54mm_Vertical footprint, which includes a bundled
STEP 3D model - no fork needed, pin numbering (1-20) matches exactly.

Official footprint anchors at pad1 (local origin) with pads running
along local +Y, versus the project's original center-anchored,
90°-rotated instance. Solved for the correction via the project's
established rotation transform against pad1/pad2 world positions
(180° rotation, position (91.44, 85.09)), and verified against all
20 pads - every pad lands on its exact pre-swap world position with
unchanged net assignments (GND, ~{WR}, ~{RD}, /~{EXT_CS}, A0-A3,
D0-D7, TTL_CLK, RESET, VCC).

DRC lib_footprint_issues 30 -> 29.
Parts:
- J7: footprint My_Components:Conn_Pin_Header_20x1_2.54mm -> Connector_PinSocket_2.54mm:PinSocket_1x20_P2.54mm_Vertical
Changed lines of the file:
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@@
 			)
 		)
-		(property "Footprint" "My_Components:Conn_Pin_Header_20x1_2.54mm"
+		(property "Footprint" "Connector_PinSocket_2.54mm:PinSocket_1x20_P2.54mm_Vertical"
 			(at 40.64 55.88 0)
 			(hide yes)

Commit message: Relink U26 (IZ0512S DC-DC converter) to a materialized custom footprint
Real part is XP Power IZ0512S (Mouser 209-IZ0512S), a 3W isolated
dual +/-12V DC-DC converter in a SIP8 package with pin 4 physically
omitted (7 leads). Pulled the manufacturer's own datasheet
(SF_IZ.pdf) mechanical drawing and confirmed the project's original
pad layout (2.54mm pitch, pins 1,2,3,5,6,7,8, 17.78mm span) and pin
functions (pin7=Common, pin8=-Vout - the dual-output column) are
exactly correct.

No official KiCad footprint exists for this exact SIP8-with-pin4-
omitted package with a real 3D model - the closest official
candidates (Converter_DCDC_TRACO_TEC2/TEC3/TMR-series) reference
STEP files that don't actually exist in this KiCad 10.0.4 install,
a gap in the official library for this whole footprint family.

Built DCDC_Custom:IZ0512S instead: pads match the verified real
layout, and the 3D model is the manufacturer's own STEP model for
the related sibling part IA0512S (same SIP potted-module
construction, sourced via SamacSys/Ultra Librarian), anisotropically
scaled (1.1321x, 1.0990y, 1.5333z) from the IA0512S's real body
(19.3 x 10.1 x 6.0mm per SF_IA.pdf) to the IZ0512S's real body
(21.85 x 11.10 x 9.20mm per SF_IZ.pdf). This is a documented
approximation, not an exact manufacturer model, since none exists
for this exact part.

New footprint anchors at pad1 (local origin) with pads running
along local +X, so no board rotation was needed - only a position
correction (68.58, 10.16) to match the pre-swap pad1 world location.
Verified all 7 pads land exactly on their pre-swap positions with
unchanged net assignments (GND, VCC, +12V, -12V, and the two
no-connect nets).

DRC lib_footprint_issues 28 -> 27.
Parts:
- U26: footprint My_Components:DC-DC_SIP8 -> DCDC_Custom:IZ0512S
Changed lines of the file:
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@@
 			)
 		)
-		(property "Footprint" "My_Components:DC-DC_SIP8"
+		(property "Footprint" "DCDC_Custom:IZ0512S"
 			(at 66.04 153.67 0)
 			(hide yes)

Commit message: Relink U25 (LM7905 -5V regulator) to the official footprint
Real part is LM7905CT-NOPB (Mouser 926-LM7905CT-NOPB), a standard
TO-220-3 negative linear regulator. Relinked to the official
Package_TO_SOT_THT:TO-220-3_Vertical footprint, which includes a
bundled STEP 3D model. Pad pitch (2.54mm) matches exactly; pad/drill
size is a closer fit to real TO-220 leads (1.905x2mm/1.1mm vs. the
original's 1.778mm/1.016mm).

Official footprint anchors at pad1 (local origin) versus the
project's center-pin-anchored instance, but both use the same
local +X pad-index direction, so only a position correction was
needed (48.26, 8.89 = old pad1 world location), no rotation change.
Verified all 3 pads land exactly on their pre-swap world positions,
nets unchanged (GND, -12V, -5V).

DRC lib_footprint_issues 27 -> 26.
Parts:
- U25: footprint My_Components:IC_TO220-3_Vert -> Package_TO_SOT_THT:TO-220-3_Vertical
Changed lines of the file:
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@@
 			)
 		)
-		(property "Footprint" "My_Components:IC_TO220-3_Vert"
+		(property "Footprint" "Package_TO_SOT_THT:TO-220-3_Vertical"
 			(at 152.4 111.76 0)
 			(hide yes)
