File: KiCad/Radio-86RK-Power.kicad_sch (KiCad schematic)
At the start: 52 parts, among them J2 5V, J3 Power, J7 Extension, U16 7486/К155ЛП5, U17 7474/К155ТМ2, U18 7408/К155ЛИ1, U19 7404/К155ЛН1, U20 7400/К155ЛА3, U25 LM7905/КР1179ЕН5В, U26 IZ0512S

Commit message: Relink U15-U20 (14-pin DIP 74LS-series logic) to the socket+chip composite footprint
Package width confirmed 300mil DIP-14 for the 74LS family (SN74LS00N: TI "N
package" PDIP-14), matching the board's existing 7.62mm row spacing. Reuses
the Task 23 IC_Socket_Custom compositing approach: pads/silkscreen from the
official Package_DIP:DIP-14_W7.62mm_Socket footprint, plus two composited
3D models (official socket STEP at board level, official chip STEP raised
5.48mm - real stack height of the BOM socket, Mouser 649-DILB14P-223TLF).

All 6 references are multi-unit symbols with redundant per-unit Footprint
property copies spread across up to 4 sheet files each (26 unit-instance
copies total) - batch_edit_schematic_components only patches one instance
per reference per call, so remaining stragglers were located and verified
by reference before a direct text substitution.

Anchor point moved from array-center to pad1 and rotation recomputed
180 (from F8's preserved 90) per instance, verified: all six show the
correct universal 74-series DIP-14 power pinout (pad7=GND, pad14=VCC),
and U15's full pad/net list matches the pre-swap board exactly.

Co-Authored-By: Claude Sonnet 5 <noreply@anthropic.com>
Parts:
- U16, U17, U18, U19, U20: footprint My_Components:IC_DIP14_300 -> IC_Socket_Custom:DIP-14_W7.62mm_Socketed
Changed lines of the file:
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@@
 			)
 		)
-		(property "Footprint" "My_Components:IC_DIP14_300"
+		(property "Footprint" "IC_Socket_Custom:DIP-14_W7.62mm_Socketed"
 			(at 172.72 142.24 0)
 			(hide yes)
@@
 			)
 		)
-		(property "Footprint" "My_Components:IC_DIP14_300"
+		(property "Footprint" "IC_Socket_Custom:DIP-14_W7.62mm_Socketed"
 			(at 187.96 142.24 0)
 			(hide yes)
@@
 			)
 		)
-		(property "Footprint" "My_Components:IC_DIP14_300"
+		(property "Footprint" "IC_Socket_Custom:DIP-14_W7.62mm_Socketed"
 			(at 157.48 142.24 0)
 			(hide yes)
@@
 			)
 		)
-		(property "Footprint" "My_Components:IC_DIP14_300"
+		(property "Footprint" "IC_Socket_Custom:DIP-14_W7.62mm_Socketed"
 			(at 127 142.24 0)
 			(hide yes)
@@
 			)
 		)
-		(property "Footprint" "My_Components:IC_DIP14_300"
+		(property "Footprint" "IC_Socket_Custom:DIP-14_W7.62mm_Socketed"
 			(at 142.24 142.24 0)
 			(hide yes)
