File: KiCad/Radio-86RK-Power.kicad_sch (KiCad schematic)
At the start: 52 parts, among them J2 5V, J3 Power, J7 Extension, U16 7486/К155ЛП5, U17 7474/К155ТМ2, U18 7408/К155ЛИ1, U19 7404/К155ЛН1, U20 7400/К155ЛА3, U25 LM7905/КР1179ЕН5В, U26 IZ0512S

Commit message: Re-home HOLE (mounting-hole placeholder) from lost my_components library
First step of an 18-commit, part-by-part redo of the "Re-home 27
components" relink (previously done as a single monolithic commit that
silently dropped two symbols' mirror transforms — see plan doc). Creates
the project-local Radio86RK_Custom.kicad_sym library and registers it via
sym-lib-table, seeded with just the HOLE symbol definition extracted
byte-for-byte from the schematic's own embedded cache. Relinks HOLE1-7 on
the Power sheet from my_components:HOLE to Radio86RK_Custom:HOLE.

ERC: 52 violations / 0 errors (no new errors introduced).
Parts:
- HOLE1, HOLE2, HOLE3, HOLE4, HOLE5, HOLE6, HOLE7: symbol my_components:HOLE -> Radio86RK_Custom:HOLE
Changed lines of the file:
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@@
 	)
 	(symbol
-		(lib_id "my_components:HOLE")
+		(lib_id "Radio86RK_Custom:HOLE")
 		(at 262.89 76.2 0)
 		(unit 1)
@@
 	)
 	(symbol
-		(lib_id "my_components:HOLE")
+		(lib_id "Radio86RK_Custom:HOLE")
 		(at 262.89 81.28 0)
 		(unit 1)
@@
 	)
 	(symbol
-		(lib_id "my_components:HOLE")
+		(lib_id "Radio86RK_Custom:HOLE")
 		(at 262.89 86.36 0)
 		(unit 1)
@@
 	)
 	(symbol
-		(lib_id "my_components:HOLE")
+		(lib_id "Radio86RK_Custom:HOLE")
 		(at 262.89 91.44 0)
 		(unit 1)
@@
 	)
 	(symbol
-		(lib_id "my_components:HOLE")
+		(lib_id "Radio86RK_Custom:HOLE")
 		(at 262.89 96.52 0)
 		(unit 1)
@@
 	)
 	(symbol
-		(lib_id "my_components:HOLE")
+		(lib_id "Radio86RK_Custom:HOLE")
 		(at 262.89 101.6 0)
 		(unit 1)
@@
 	)
 	(symbol
-		(lib_id "my_components:HOLE")
+		(lib_id "Radio86RK_Custom:HOLE")
 		(at 262.89 106.68 0)
 		(unit 1)

Commit message: Re-home IZ0512S (DC-DC converter) from lost my_components library
Step 2/18 of the part-by-part redo. Relinks U26 on the Power sheet from
my_components:IZ0512S to Radio86RK_Custom:IZ0512S.
Parts:
- U26: symbol my_components:IZ0512S -> Radio86RK_Custom:IZ0512S
Changed lines of the file:
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@@
 	)
 	(symbol
-		(lib_id "my_components:IZ0512S")
+		(lib_id "Radio86RK_Custom:IZ0512S")
 		(at 66.04 144.78 0)
 		(unit 1)
