File: KiCad/Radio-86RK-Keyboard.kicad_sch (KiCad schematic)
At the start: 96 parts, among them J4 Cassette, SW1 FF, SW10 LF ПС, SW11 CR ВК, SW12 DEL ЗБ, SW13 LEFT, SW14 UP, SW15 RIGHT, SW16 DOWN, SW17 0, SW18 1 !, SW19 2 ", SW2 CLS СТР, SW20 3 #, SW21 4 $, SW22 5 %, SW23 6 &, SW24 7 ', SW25 8 (, SW26 9 ), SW27 : *, SW28 ; +, SW29 , <, SW3 ESC АР2, SW30 - =, SW31 . >, SW32 / ?, SW33 @ Ю, SW34 A А, SW35 B Б, SW36 C Ц, SW37 D Д, SW38 E Е, SW39 F Ф, SW4 F1, SW40 G Г, SW41 H Х, SW42 I И, SW43 J Й, SW44 K К, SW45 L Л, SW46 M М, SW47 N Н, SW48 O О, SW49 P П, SW5 F2, SW50 Q Я, SW51 R Р, SW52 S С, SW53 T Т, SW54 U У, SW55 V Ж, SW56 W В, SW57 X Ь, SW58 Y Ы, SW59 Z З, SW6 F3, SW60 [ Ш, SW61 \ Э, SW62 ] Щ, SW63 ^ Ч, SW64 SPACE, SW65 CTRL УС, SW66 SHIFT CC, SW67 RUS/LAT, SW7 F4, SW8 F5, SW9 TAB ТАБ, U19 7404/К155ЛН1, U21 TL071/КР140УД608, U5 8255A/КР580ВВ55А

Commit message: Fix broken Cherry_MX footprint library link for 65 keyboard switches
The Cherry_MX nickname referenced by SW1-SW67 footprints had no fp-lib-table
entry anywhere (project or global), so DRC flagged 'library not found' for
every switch. Added a project-local fp-lib-table registering Cherry_MX
against the PCM-installed keyswitch-kicad-library, and relinked the 65
switches using standard 1.00u/1.25u/1.50u footprints to the matching
official SW_Cherry_MX_PCB_* footprints (pad layout is equivalent, only
mil- vs metric-rounded).

SW11 (Enter, 2.25u) and SW64 (Space, 6.25u) are intentionally left on
their original footprints: the official 2.25u/6.25u footprints lack the
stabilizer mounting holes that this project's legacy footprints have, so
swapping them would remove real hardware (stabilizer wire mounts).

Co-Authored-By: Claude Sonnet 5 <noreply@anthropic.com>
Parts:
- SW1, SW10, SW12, SW13, SW14, SW15, SW16, SW17, SW18, SW19, SW2, SW20, SW21, SW22, SW23, SW24, SW25, SW26, SW27, SW28, SW29, SW3, SW30, SW31, SW32, SW33, SW34, SW35, SW36, SW37, SW38, SW39, SW4, SW40, SW41, SW42, SW43, SW44, SW45, SW46, SW47, SW48, SW49, SW5, SW50, SW51, SW52, SW53, SW54, SW55, SW56, SW57, SW58, SW59, SW6, SW60, SW62, SW63, SW67, SW7, SW8, SW9: footprint Cherry_MX:CHERRY_PCB_100H -> Cherry_MX:SW_Cherry_MX_PCB_1.00u
- SW61: footprint Cherry_MX:CHERRY_PCB_150H -> Cherry_MX:SW_Cherry_MX_PCB_1.50u
- SW65, SW66: footprint Cherry_MX:CHERRY_PCB_125H -> Cherry_MX:SW_Cherry_MX_PCB_1.25u

Commit message: Link SW11/SW64 to custom Cherry MX footprints with stabilizer 3D models
SW11 (Enter, 2.25u) and SW64 (Space, 6.25u) use a hand-built leveling
kit (Mouser 540-G99-0742 + 540-G99-0226, per README BOM) with no
matching footprint in the official keyswitch-kicad-library, so they
were left unlinked when the other 65 switches were relinked to the
official Cherry_MX library.

Extracted their exact existing 9-pad geometry from the PCB into a new
project-local Cherry_MX_Custom.pretty library (self-contained, no
external dependency), registered via a second fp-lib-table entry, and
pointed both schematic symbols at it.

Also attached 3D models: the switch body (shared with the other 65
switches) plus the closest-matching official stabilizer model for
each (Stabilizer_Cherry_MX_2.00u for Enter, 6.25u for Space) - their
hole spacing matches this project's embedded geometry almost exactly,
confirmed pad-by-pad. Needed for accurate mechanical reference when
modeling the case in FreeCAD.

Co-Authored-By: Claude Sonnet 5 <noreply@anthropic.com>
Parts:
- SW11: footprint Cherry_MX:CHERRY_PCB_225H -> Cherry_MX_Custom:CHERRY_PCB_225H
- SW64: footprint Cherry_MX:CHERRY_PCB_625H -> Cherry_MX_Custom:CHERRY_PCB_625H
Changed lines of the file:
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@@
 		)
 		(property "Intersheetrefs" "${INTERSHEET_REFS}"
-			(at 0 0 0)
+			(at 243.84 97.5695 90)
 			(hide yes)
 			(show_name no)
@@
 					(size 1.27 1.27)
 				)
+				(justify left)
 			)
 		)
@@
 		)
 		(property "Intersheetrefs" "${INTERSHEET_REFS}"
-			(at 0 0 0)
+			(at 19.8455 114.3 0)
 			(hide yes)
 			(show_name no)
@@
 					(size 1.27 1.27)
 				)
+				(justify right)
 			)
 		)
@@
 		)
 		(property "Intersheetrefs" "${INTERSHEET_REFS}"
-			(at 0 0 0)
+			(at 15.7089 137.16 0)
 			(hide yes)
 			(show_name no)
@@
 					(size 1.27 1.27)
 				)
+				(justify right)
 			)
 		)
@@
 		)
 		(property "Intersheetrefs" "${INTERSHEET_REFS}"
-			(at 0 0 0)
+			(at 18.4848 86.36 0)
 			(hide yes)
 			(show_name no)
@@
 					(size 1.27 1.27)
 				)
+				(justify right)
 			)
 		)
@@
 		)
 		(property "Intersheetrefs" "${INTERSHEET_REFS}"
-			(at 0 0 0)
+			(at 18.4848 99.06 0)
 			(hide yes)
 			(show_name no)
@@
 					(size 1.27 1.27)
 				)
+				(justify right)
 			)
 		)
@@
 		)
 		(property "Intersheetrefs" "${INTERSHEET_REFS}"
-			(at 0 0 0)
+			(at 18.4848 88.9 0)
 			(hide yes)
 			(show_name no)
@@
 					(size 1.27 1.27)
 				)
+				(justify right)
 			)
 		)
@@
 		)
 		(property "Intersheetrefs" "${INTERSHEET_REFS}"
-			(at 0 0 0)
+			(at 19.3375 132.08 0)
 			(hide yes)
 			(show_name no)
@@
 					(size 1.27 1.27)
 				)
+				(justify right)
 			)
 		)
@@
 		)
 		(property "Intersheetrefs" "${INTERSHEET_REFS}"
-			(at 0 0 0)
+			(at 19.8455 116.84 0)
 			(hide yes)
 			(show_name no)
@@
 					(size 1.27 1.27)
 				)
+				(justify right)
 			)
 		)
@@
 		)
 		(property "Intersheetrefs" "${INTERSHEET_REFS}"
-			(at 0 0 0)
+			(at 18.4848 93.98 0)
 			(hide yes)
 			(show_name no)
@@
 					(size 1.27 1.27)
 				)
+				(justify right)
 			)
 		)
@@
 		)
 		(property "Intersheetrefs" "${INTERSHEET_REFS}"
-			(at 0 0 0)
+			(at 18.4848 96.52 0)
 			(hide yes)
 			(show_name no)
@@
 					(size 1.27 1.27)
 				)
+				(justify right)
 			)
 		)
@@
 		)
 		(property "Intersheetrefs" "${INTERSHEET_REFS}"
-			(at 0 0 0)
+			(at 12.2981 165.1 0)
 			(hide yes)
 			(show_name no)
@@
 					(size 1.27 1.27)
 				)
+				(justify right)
 			)
 		)
@@
 		)
 		(property "Intersheetrefs" "${INTERSHEET_REFS}"
-			(at 0 0 0)
+			(at 248.92 98.513 90)
 			(hide yes)
 			(show_name no)
@@
 					(size 1.27 1.27)
 				)
+				(justify left)
 			)
 		)
@@
 		)
 		(property "Intersheetrefs" "${INTERSHEET_REFS}"
-			(at 0 0 0)
+			(at 18.4848 101.6 0)
 			(hide yes)
 			(show_name no)
@@
 					(size 1.27 1.27)
 				)
+				(justify right)
 			)
 		)
@@
 		)
 		(property "Intersheetrefs" "${INTERSHEET_REFS}"
-			(at 0 0 0)
+			(at 19.5552 127 0)
 			(hide yes)
 			(show_name no)
@@
 					(size 1.27 1.27)
 				)
+				(justify right)
 			)
 		)
@@
 		)
 		(property "Intersheetrefs" "${INTERSHEET_REFS}"
-			(at 0 0 0)
+			(at 18.4848 104.14 0)
 			(hide yes)
 			(show_name no)
@@
 					(size 1.27 1.27)
 				)
+				(justify right)
 			)
 		)
@@
 		)
 		(property "Intersheetrefs" "${INTERSHEET_REFS}"
-			(at 0 0 0)
+			(at 11.1369 170.18 0)
 			(hide yes)
 			(show_name no)
@@
 					(size 1.27 1.27)
 				)
+				(justify right)
 			)
 		)
@@
 		)
 		(property "Intersheetrefs" "${INTERSHEET_REFS}"
-			(at 0 0 0)
+			(at 18.4848 91.44 0)
 			(hide yes)
 			(show_name no)
@@
 					(size 1.27 1.27)
 				)
+				(justify right)
 			)
 		)
@@
 			)
 		)
-		(property "Footprint" "Cherry_MX:CHERRY_PCB_225H"
+		(property "Footprint" "Cherry_MX_Custom:CHERRY_PCB_225H"
 			(at 154.94 35.56 0)
 			(hide yes)
@@
 			)
 		)
-		(property "Footprint" "Cherry_MX:CHERRY_PCB_625H"
+		(property "Footprint" "Cherry_MX_Custom:CHERRY_PCB_625H"
 			(at 231.14 111.76 0)
 			(hide yes)

Commit message: Relink R1-R15 to official Resistor_THT footprint
The 15 discrete resistors used My_Components:Res_762, an unresolved
library nickname with no fp-lib-table entry anywhere on disk. Compared
the footprint against the actual ordered part (Stackpole CF14 1/4W
carbon film, per the README Mouser BOM) rather than just the closest
official name: the real part's datasheet body (6.50x2.30mm) is closer
to Resistor_THT:R_Axial_DIN0207_L6.3mm_D2.5mm_P7.62mm_Horizontal's
silkscreen outline (6.54x2.74mm) than to the project's own hand-drawn
one (5.84x2.03mm), so the official footprint is the more accurate
choice, not just a fallback. Same 7.62mm pin pitch, and it comes with
a working 3D model - the project's own model reference
("discret/resistor.wrl") doesn't resolve on any current KiCad install.

Co-Authored-By: Claude Sonnet 5 <noreply@anthropic.com>
Parts:
- R12, R13, R14, R15, R4, R7, R8: footprint My_Components:Res_762 -> Resistor_THT:R_Axial_DIN0207_L6.3mm_D2.5mm_P7.62mm_Horizontal
Changed lines of the file:
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@@
 			)
 		)
-		(property "Footprint" "My_Components:Res_762"
+		(property "Footprint" "Resistor_THT:R_Axial_DIN0207_L6.3mm_D2.5mm_P7.62mm_Horizontal"
 			(at 80.01 49.022 90)
 			(hide yes)
@@
 			)
 		)
-		(property "Footprint" "My_Components:Res_762"
+		(property "Footprint" "Resistor_THT:R_Axial_DIN0207_L6.3mm_D2.5mm_P7.62mm_Horizontal"
 			(at 80.01 38.862 90)
 			(hide yes)
@@
 			)
 		)
-		(property "Footprint" "My_Components:Res_762"
+		(property "Footprint" "Resistor_THT:R_Axial_DIN0207_L6.3mm_D2.5mm_P7.62mm_Horizontal"
 			(at 43.18 181.102 90)
 			(hide yes)
@@
 			)
 		)
-		(property "Footprint" "My_Components:Res_762"
+		(property "Footprint" "Resistor_THT:R_Axial_DIN0207_L6.3mm_D2.5mm_P7.62mm_Horizontal"
 			(at 54.102 189.23 90)
 			(hide yes)
@@
 			)
 		)
-		(property "Footprint" "My_Components:Res_762"
+		(property "Footprint" "Resistor_THT:R_Axial_DIN0207_L6.3mm_D2.5mm_P7.62mm_Horizontal"
 			(at 94.742 189.23 90)
 			(hide yes)
@@
 			)
 		)
-		(property "Footprint" "My_Components:Res_762"
+		(property "Footprint" "Resistor_THT:R_Axial_DIN0207_L6.3mm_D2.5mm_P7.62mm_Horizontal"
 			(at 112.522 189.23 90)
 			(hide yes)
@@
 			)
 		)
-		(property "Footprint" "My_Components:Res_762"
+		(property "Footprint" "Resistor_THT:R_Axial_DIN0207_L6.3mm_D2.5mm_P7.62mm_Horizontal"
 			(at 143.51 178.562 90)
 			(hide yes)

Commit message: Relink ceramic capacitors and F1 polyfuse to official footprints
The 39 refs (C1-C32, C39-C44, F1) used My_Components:Cap_Cer_508, an
unresolved library nickname. Resolved the real ordered parts from the
README Mouser BOM: C1-C32 are Vishay K104K15X7RF53H5 (~4.0x4.0x2.6mm
body), C40-C44 are TDK FG28-series (~4.0x5.5mm body), C39 is TDK
FG24-series (~4.5x5.5mm, larger), and F1 is a Littelfuse 16R110BU PTC
resettable fuse with no dedicated KiCad footprint.

All share the project's existing 5.08mm pitch (matches every
datasheet's 5.0mm +/-0.8-1.0mm spec). Split into two official
Capacitor_THT footprints matching the two real body-size groups
(C_Disc_D4.7mm_W2.5mm_P5.00mm for the smaller Vishay/FG28 parts,
C_Disc_D5.1mm_W3.2mm_P5.00mm for the larger FG24 C39) rather than
forcing one footprint on parts of two different real sizes. F1 reuses
the small-cap disc footprint since Littelfuse's radial PTC package at
this pitch is mechanically a disc shape with no official equivalent.

Co-Authored-By: Claude Sonnet 5 <noreply@anthropic.com>
Parts:
- C31, C32, C42: footprint My_Components:Cap_Cer_508 -> Capacitor_THT:C_Disc_D4.7mm_W2.5mm_P5.00mm
- C39: footprint My_Components:Cap_Cer_508 -> Capacitor_THT:C_Disc_D5.1mm_W3.2mm_P5.00mm
Changed lines of the file:
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@@
 			)
 		)
-		(property "Footprint" "My_Components:Cap_Cer_508"
+		(property "Footprint" "Capacitor_THT:C_Disc_D4.7mm_W2.5mm_P5.00mm"
 			(at 49.8348 185.42 0)
 			(hide yes)
@@
 			)
 		)
-		(property "Footprint" "My_Components:Cap_Cer_508"
+		(property "Footprint" "Capacitor_THT:C_Disc_D4.7mm_W2.5mm_P5.00mm"
 			(at 58.42 183.8452 0)
 			(hide yes)
@@
 			)
 		)
-		(property "Footprint" "My_Components:Cap_Cer_508"
+		(property "Footprint" "Capacitor_THT:C_Disc_D5.1mm_W3.2mm_P5.00mm"
 			(at 106.68 181.9148 0)
 			(hide yes)
@@
 			)
 		)
-		(property "Footprint" "My_Components:Cap_Cer_508"
+		(property "Footprint" "Capacitor_THT:C_Disc_D4.7mm_W2.5mm_P5.00mm"
 			(at 108.2548 193.04 0)
 			(hide yes)

Commit message: Relink diodes D1-D9 to official DO-35 footprint
Real part is 1N4148 (DO-35 package, ~4.25-4.6mm body, ~1.85-2mm
diameter). Diode_THT:D_DO-35_SOD27_P7.62mm_Horizontal is an exact
pitch match; confirmed pad 1 = cathode in both the project's original
footprint (via its embedded pinfunction "K_1"/"A_2" metadata) and the
official library file, so the swap carries no polarity risk.

Note: the PCB-side footprint swap and the resulting placement-anchor
correction for D1-D9 already landed in the previous commit
(967499e) together with the retroactive fix for R1-R15 and the
capacitors, since all of it was discovered and fixed in the same
pass. This commit is just the schematic-side Footprint field change.

Co-Authored-By: Claude Sonnet 5 <noreply@anthropic.com>
Parts:
- D1, D2, D3, D4, D5, D6, D7, D8, D9: footprint My_Components:Diode_762 -> Diode_THT:D_DO-35_SOD27_P7.62mm_Horizontal
Changed lines of the file:
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@@
 			)
 		)
-		(property "Footprint" "My_Components:Diode_762"
+		(property "Footprint" "Diode_THT:D_DO-35_SOD27_P7.62mm_Horizontal"
 			(at 115.57 30.48 0)
 			(hide yes)
@@
 			)
 		)
-		(property "Footprint" "My_Components:Diode_762"
+		(property "Footprint" "Diode_THT:D_DO-35_SOD27_P7.62mm_Horizontal"
 			(at 115.57 43.18 0)
 			(hide yes)
@@
 			)
 		)
-		(property "Footprint" "My_Components:Diode_762"
+		(property "Footprint" "Diode_THT:D_DO-35_SOD27_P7.62mm_Horizontal"
 			(at 115.57 55.88 0)
 			(hide yes)
@@
 			)
 		)
-		(property "Footprint" "My_Components:Diode_762"
+		(property "Footprint" "Diode_THT:D_DO-35_SOD27_P7.62mm_Horizontal"
 			(at 115.57 17.78 0)
 			(hide yes)
@@
 			)
 		)
-		(property "Footprint" "My_Components:Diode_762"
+		(property "Footprint" "Diode_THT:D_DO-35_SOD27_P7.62mm_Horizontal"
 			(at 115.57 81.28 0)
 			(hide yes)
@@
 			)
 		)
-		(property "Footprint" "My_Components:Diode_762"
+		(property "Footprint" "Diode_THT:D_DO-35_SOD27_P7.62mm_Horizontal"
 			(at 115.57 93.98 0)
 			(hide yes)
@@
 			)
 		)
-		(property "Footprint" "My_Components:Diode_762"
+		(property "Footprint" "Diode_THT:D_DO-35_SOD27_P7.62mm_Horizontal"
 			(at 115.57 106.68 0)
 			(hide yes)
@@
 			)
 		)
-		(property "Footprint" "My_Components:Diode_762"
+		(property "Footprint" "Diode_THT:D_DO-35_SOD27_P7.62mm_Horizontal"
 			(at 115.57 68.58 0)
 			(hide yes)
@@
 			)
 		)
-		(property "Footprint" "My_Components:Diode_762"
+		(property "Footprint" "Diode_THT:D_DO-35_SOD27_P7.62mm_Horizontal"
 			(at 149.86 186.69 0)
 			(hide yes)

Commit message: Relink LEDs D10/D11 to official 3mm THT footprint
Real parts are Broadcom HLMP-1503 (green) / HLMP-1401 (yellow), T-1
(3mm) diffused lamps - confirmed 3.17mm max body diameter and standard
2.54mm lead pitch matching the project exactly.
LED_THT:LED_D3.0mm is an exact match; pad 1 = rect = cathode in both
the official footprint and the project's original (via its GND net
assignment), so no polarity risk.

The project's original footprint had pad1 on the opposite side from
the official convention (same class of inversion as the diodes),
requiring a +180 degree rotation correction in addition to the
position shift - applied and verified immediately this time (pad
positions and net mappings confirmed identical to pre-swap; DRC
lib_footprint_issues 51->49, no dangling-track/thermal regressions).

Co-Authored-By: Claude Sonnet 5 <noreply@anthropic.com>
Parts:
- D10, D11: footprint My_Components:LED_3mm -> LED_THT:LED_D3.0mm
Changed lines of the file:
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@@
 			)
 		)
-		(property "Footprint" "My_Components:LED_3mm"
+		(property "Footprint" "LED_THT:LED_D3.0mm"
 			(at 62.23 40.64 0)
 			(hide yes)
@@
 			)
 		)
-		(property "Footprint" "My_Components:LED_3mm"
+		(property "Footprint" "LED_THT:LED_D3.0mm"
 			(at 62.23 50.8 0)
 			(hide yes)

Commit message: Relink RN2-RN4 (4.7k SIP6 resistor arrays) to official footprint
Real part is Bourns 4606X, bussed SIP6 topology (1 common pin + 5
resistors), 2.54mm pitch - matches existing wiring exactly (pad 1 =
VCC common bus). Resistor_THT:R_Array_SIP6 is an exact pitch/
convention match.

Note on this task's process: the position-correction move_component
calls were initially applied before the schematic-side footprint swap
had actually been forward-annotated and saved to the PCB on disk (the
MCP backend session was reading a stale cached copy even after
reopening), so the first correction attempt was computed against the
still-old centered-anchor footprint and produced a wrong result. Reverted
to the true original position, waited for confirmation the PCB was
actually saved, then reapplied the same (correct) formula successfully.
All 6 pads per reference verified identical to pre-swap.

Co-Authored-By: Claude Sonnet 5 <noreply@anthropic.com>
Parts:
- RN2, RN3, RN4: footprint My_Components:Conn_SIL6 -> Resistor_THT:R_Array_SIP6
Changed lines of the file:
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@@
 			)
 		)
-		(property "Footprint" "My_Components:Conn_SIL6"
+		(property "Footprint" "Resistor_THT:R_Array_SIP6"
 			(at 256.54 151.765 90)
 			(hide yes)
@@
 			)
 		)
-		(property "Footprint" "My_Components:Conn_SIL6"
+		(property "Footprint" "Resistor_THT:R_Array_SIP6"
 			(at 212.09 164.465 90)
 			(hide yes)
@@
 			)
 		)
-		(property "Footprint" "My_Components:Conn_SIL6"
+		(property "Footprint" "Resistor_THT:R_Array_SIP6"
 			(at 256.54 128.905 90)
 			(hide yes)

Commit message: Relink J4 (8-pin right-angle DIN jack) to a materialized custom footprint
My_Components:Conn_DIN_8pin had no official KiCad match: the only
DIN-related library (Connector_DIN) contains exclusively rectangular
DIN41612 card-edge connectors, unrelated to a round 8-pin DIN socket.

Sourced the manufacturer's own KiCad export (SamacSys/Ultra
Librarian) for the exact real part (Same Sky/CUI SDF-80J, Mouser
490-SDF-80J), registered as Conn_DIN_Custom:SDF-80J. Verified the
12-pad geometry is a clean 180 degree rotation of the project's
existing layout (confirmed pad-by-pad, including the 2 large
mechanical pads and 2 small shield-tab pads, not just the 8 signal
pins), then renamed the manufacturer's MH1-MH4 mechanical pads to
match the project's schematic-driven pad naming ('~' for the two
unconnected mounting legs, '0' for the two GND shield tabs sharing a
single symbol pin) so the existing net wiring carries over unchanged.
Includes the manufacturer's STEP 3D model.

Corrected the anchor-point/rotation after forward-annotation: moved
to (97.87, 19.05) and rotated 180 degrees. All 12 pads now land
exactly on their pre-swap world positions with unchanged net
assignments. 3D model orientation verified visually.

Co-Authored-By: Claude Sonnet 5 <noreply@anthropic.com>
Parts:
- J4: footprint My_Components:Conn_DIN_8pin -> Conn_DIN_Custom:SDF-80J
Changed lines of the file:
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@@
 			)
 		)
-		(property "Footprint" "My_Components:Conn_DIN_8pin"
+		(property "Footprint" "Conn_DIN_Custom:SDF-80J"
 			(at 81.28 185.42 0)
 			(hide yes)
