File: KiCad/Radio-86RK-Keyboard.kicad_sch (KiCad schematic)
At the start: 96 parts, among them J4 Cassette, SW1 FF, SW10 LF ПС, SW11 CR ВК, SW12 DEL ЗБ, SW13 LEFT, SW14 UP, SW15 RIGHT, SW16 DOWN, SW17 0, SW18 1 !, SW19 2 ", SW2 CLS СТР, SW20 3 #, SW21 4 $, SW22 5 %, SW23 6 &, SW24 7 ', SW25 8 (, SW26 9 ), SW27 : *, SW28 ; +, SW29 , <, SW3 ESC АР2, SW30 - =, SW31 . >, SW32 / ?, SW33 @ Ю, SW34 A А, SW35 B Б, SW36 C Ц, SW37 D Д, SW38 E Е, SW39 F Ф, SW4 F1, SW40 G Г, SW41 H Х, SW42 I И, SW43 J Й, SW44 K К, SW45 L Л, SW46 M М, SW47 N Н, SW48 O О, SW49 P П, SW5 F2, SW50 Q Я, SW51 R Р, SW52 S С, SW53 T Т, SW54 U У, SW55 V Ж, SW56 W В, SW57 X Ь, SW58 Y Ы, SW59 Z З, SW6 F3, SW60 [ Ш, SW61 \ Э, SW62 ] Щ, SW63 ^ Ч, SW64 SPACE, SW65 CTRL УС, SW66 SHIFT CC, SW67 RUS/LAT, SW7 F4, SW8 F5, SW9 TAB ТАБ, U19 7404/К155ЛН1, U21 TL071/КР140УД608, U5 8255A/КР580ВВ55А

Commit message: Relink U21/U23/U24 (8-pin DIP ICs) to a materialized socket+chip composite footprint
Package width confirmed 300mil DIP-8 against TL071 (TI: "P (PDIP, 8)") and
SN75150P (TI: "P PDIP 8", 13.97mm tube width) datasheets, matching the
board's existing 7.62mm row spacing.

New IC_Socket_Custom:DIP-8_W7.62mm_Socketed footprint reuses the official
Package_DIP:DIP-8_W7.62mm_Socket pads/silkscreen, with two composited 3D
models: the official socket STEP at board level plus the official bare-chip
STEP raised 5.1mm in Z (real stack height of the BOM socket, Mouser
649-DILB8P223TLF) so the chip renders seated in its socket. Both models are
official KiCad Package_DIP assets - no missing-model gap this time.

Anchor point moved from array-center (old hand-drawn footprint) to pad1
(official footprint convention); required rotation recomputed from scratch
per-instance (90 -> 180) rather than trusting F8's preserved old rotation
value, verified against all 8 pads/nets per instance before committing.

Co-Authored-By: Claude Sonnet 5 <noreply@anthropic.com>
Parts:
- U21: footprint My_Components:IC_DIP8_300 -> IC_Socket_Custom:DIP-8_W7.62mm_Socketed
Changed lines of the file:
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@@
 			)
 		)
-		(property "Footprint" "My_Components:IC_DIP8_300"
+		(property "Footprint" "IC_Socket_Custom:DIP-8_W7.62mm_Socketed"
 			(at 130.81 175.26 0)
 			(hide yes)

Commit message: Relink U15-U20 (14-pin DIP 74LS-series logic) to the socket+chip composite footprint
Package width confirmed 300mil DIP-14 for the 74LS family (SN74LS00N: TI "N
package" PDIP-14), matching the board's existing 7.62mm row spacing. Reuses
the Task 23 IC_Socket_Custom compositing approach: pads/silkscreen from the
official Package_DIP:DIP-14_W7.62mm_Socket footprint, plus two composited
3D models (official socket STEP at board level, official chip STEP raised
5.48mm - real stack height of the BOM socket, Mouser 649-DILB14P-223TLF).

All 6 references are multi-unit symbols with redundant per-unit Footprint
property copies spread across up to 4 sheet files each (26 unit-instance
copies total) - batch_edit_schematic_components only patches one instance
per reference per call, so remaining stragglers were located and verified
by reference before a direct text substitution.

Anchor point moved from array-center to pad1 and rotation recomputed
180 (from F8's preserved 90) per instance, verified: all six show the
correct universal 74-series DIP-14 power pinout (pad7=GND, pad14=VCC),
and U15's full pad/net list matches the pre-swap board exactly.

Co-Authored-By: Claude Sonnet 5 <noreply@anthropic.com>
Parts:
- U19: footprint My_Components:IC_DIP14_300 -> IC_Socket_Custom:DIP-14_W7.62mm_Socketed
Changed lines of the file:
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@@
 			)
 		)
-		(property "Footprint" "My_Components:IC_DIP14_300"
+		(property "Footprint" "IC_Socket_Custom:DIP-14_W7.62mm_Socketed"
 			(at 35.56 40.64 0)
 			(hide yes)

Commit message: Relink U1/U5/U6/U7/U8 (40-pin DIP ICs) to the socket+chip composite footprint
Package width confirmed 600mil DIP-40 - the board's own measured 15.24mm row
spacing already matched Package_DIP:DIP-40_W15.24mm exactly, and the Intel
8080A/8255A/8257/8275 family is universally packaged in standard 40-pin
plastic DIP with no narrow-body variant.

Reuses the Task 23 IC_Socket_Custom compositing approach: pads/silkscreen
from the official Package_DIP:DIP-40_W15.24mm_Socket footprint, plus two
composited 3D models (official socket STEP at board level, official chip
STEP raised 5.48mm - stack height directly confirmed for the BOM socket,
Mouser 649-DILB40P223TLF).

Anchor point moved from array-center to pad1 and rotation recomputed 180
(from F8's preserved 90) per instance; U1's full pad/net list matches the
pre-swap board exactly, and U5/U6/U7/U8 all show correct standard 40-pin
pinouts (GND/VCC at the expected positions).

This is the last unresolved My_Components reference in the project - DRC
confirms the "lib_footprint_issues" category has dropped to 0 (from 21
after Task 23), matching the plan's expected end state for the IC tasks.

Co-Authored-By: Claude Sonnet 5 <noreply@anthropic.com>
Parts:
- U5: footprint My_Components:IC_DIP40_600 -> IC_Socket_Custom:DIP-40_W15.24mm_Socketed
Changed lines of the file:
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@@
 			)
 		)
-		(property "Footprint" "My_Components:IC_DIP40_600"
+		(property "Footprint" "IC_Socket_Custom:DIP-40_W15.24mm_Socketed"
 			(at 50.8 118.11 0)
 			(hide yes)
