File: KiCad/Radio-86RK-Keyboard.kicad_sch (KiCad schematic)
At the start: 96 parts, among them J4 Cassette, SW1 FF, SW10 LF ПС, SW11 CR ВК, SW12 DEL ЗБ, SW13 LEFT, SW14 UP, SW15 RIGHT, SW16 DOWN, SW17 0, SW18 1 !, SW19 2 ", SW2 CLS СТР, SW20 3 #, SW21 4 $, SW22 5 %, SW23 6 &, SW24 7 ', SW25 8 (, SW26 9 ), SW27 : *, SW28 ; +, SW29 , <, SW3 ESC АР2, SW30 - =, SW31 . >, SW32 / ?, SW33 @ Ю, SW34 A А, SW35 B Б, SW36 C Ц, SW37 D Д, SW38 E Е, SW39 F Ф, SW4 F1, SW40 G Г, SW41 H Х, SW42 I И, SW43 J Й, SW44 K К, SW45 L Л, SW46 M М, SW47 N Н, SW48 O О, SW49 P П, SW5 F2, SW50 Q Я, SW51 R Р, SW52 S С, SW53 T Т, SW54 U У, SW55 V Ж, SW56 W В, SW57 X Ь, SW58 Y Ы, SW59 Z З, SW6 F3, SW60 [ Ш, SW61 \ Э, SW62 ] Щ, SW63 ^ Ч, SW64 SPACE, SW65 CTRL УС, SW66 SHIFT CC, SW67 RUS/LAT, SW7 F4, SW8 F5, SW9 TAB ТАБ, U19 7404/К155ЛН1, U21 TL071/КР140УД608, U5 8255A/КР580ВВ55А

Commit message: Re-home Conn_DIN-8 (keyboard connector) from lost my_components library
Step 11/18. Relinks J4 on the Keyboard sheet from my_components:Conn_DIN-8
to Radio86RK_Custom:Conn_DIN-8.
Parts:
- J4: symbol my_components:Conn_DIN-8 -> Radio86RK_Custom:Conn_DIN-8
Changed lines of the file:
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@@
 	)
 	(symbol
-		(lib_id "my_components:Conn_DIN-8")
+		(lib_id "Radio86RK_Custom:Conn_DIN-8")
 		(at 81.28 185.42 0)
 		(unit 1)

Commit message: Re-home 8255A (PPI) from lost my_components library
Step 12/18. Relinks U5 on the Keyboard sheet and U6 on the IO sheet from
my_components:8255A to Radio86RK_Custom:8255A (same part used on both
sheets).
Parts:
- U5: symbol my_components:8255A -> Radio86RK_Custom:8255A
Changed lines of the file:
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@@
 	)
 	(symbol
-		(lib_id "my_components:8255A")
+		(lib_id "Radio86RK_Custom:8255A")
 		(at 50.8 118.11 0)
 		(unit 1)
