File: KiCad/Radio-86RK-IO.kicad_sch (KiCad schematic)
At the start: 16 parts, among them J5 Serial, J6 Parallel, Q2 2N3904, U16 7486/К155ЛП5, U20 7400/К155ЛА3, U22 SN75154N/К170УП2В, U23 SN75150P/К170АП2, U24 SN75150P/К170АП2, U3 8251A/КР580ВВ51А, U4 8253/КР580ВИ53, U6 8255A/КР580ВВ55А

Commit message: Relink R1-R15 to official Resistor_THT footprint
The 15 discrete resistors used My_Components:Res_762, an unresolved
library nickname with no fp-lib-table entry anywhere on disk. Compared
the footprint against the actual ordered part (Stackpole CF14 1/4W
carbon film, per the README Mouser BOM) rather than just the closest
official name: the real part's datasheet body (6.50x2.30mm) is closer
to Resistor_THT:R_Axial_DIN0207_L6.3mm_D2.5mm_P7.62mm_Horizontal's
silkscreen outline (6.54x2.74mm) than to the project's own hand-drawn
one (5.84x2.03mm), so the official footprint is the more accurate
choice, not just a fallback. Same 7.62mm pin pitch, and it comes with
a working 3D model - the project's own model reference
("discret/resistor.wrl") doesn't resolve on any current KiCad install.

Co-Authored-By: Claude Sonnet 5 <noreply@anthropic.com>
Parts:
- R1, R11: footprint My_Components:Res_762 -> Resistor_THT:R_Axial_DIN0207_L6.3mm_D2.5mm_P7.62mm_Horizontal
Changed lines of the file:
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@@
 			)
 		)
-		(property "Footprint" "My_Components:Res_762"
+		(property "Footprint" "Resistor_THT:R_Axial_DIN0207_L6.3mm_D2.5mm_P7.62mm_Horizontal"
 			(at 160.782 146.05 90)
 			(hide yes)
@@
 			)
 		)
-		(property "Footprint" "My_Components:Res_762"
+		(property "Footprint" "Resistor_THT:R_Axial_DIN0207_L6.3mm_D2.5mm_P7.62mm_Horizontal"
 			(at 174.498 140.97 90)
 			(hide yes)

Commit message: Relink ceramic capacitors and F1 polyfuse to official footprints
The 39 refs (C1-C32, C39-C44, F1) used My_Components:Cap_Cer_508, an
unresolved library nickname. Resolved the real ordered parts from the
README Mouser BOM: C1-C32 are Vishay K104K15X7RF53H5 (~4.0x4.0x2.6mm
body), C40-C44 are TDK FG28-series (~4.0x5.5mm body), C39 is TDK
FG24-series (~4.5x5.5mm, larger), and F1 is a Littelfuse 16R110BU PTC
resettable fuse with no dedicated KiCad footprint.

All share the project's existing 5.08mm pitch (matches every
datasheet's 5.0mm +/-0.8-1.0mm spec). Split into two official
Capacitor_THT footprints matching the two real body-size groups
(C_Disc_D4.7mm_W2.5mm_P5.00mm for the smaller Vishay/FG28 parts,
C_Disc_D5.1mm_W3.2mm_P5.00mm for the larger FG24 C39) rather than
forcing one footprint on parts of two different real sizes. F1 reuses
the small-cap disc footprint since Littelfuse's radial PTC package at
this pitch is mechanically a disc shape with no official equivalent.

Co-Authored-By: Claude Sonnet 5 <noreply@anthropic.com>
Parts:
- C41, F1: footprint My_Components:Cap_Cer_508 -> Capacitor_THT:C_Disc_D4.7mm_W2.5mm_P5.00mm
Changed lines of the file:
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@@
 			)
 		)
-		(property "Footprint" "My_Components:Cap_Cer_508"
+		(property "Footprint" "Capacitor_THT:C_Disc_D4.7mm_W2.5mm_P5.00mm"
 			(at 129.54 194.31 0)
 			(hide yes)
@@
 			)
 		)
-		(property "Footprint" "My_Components:Cap_Cer_508"
+		(property "Footprint" "Capacitor_THT:C_Disc_D4.7mm_W2.5mm_P5.00mm"
 			(at 181.3052 157.48 0)
 			(hide yes)

Commit message: Relink transistors Q1/Q2 and U27 to official TO-92 footprint
Q1/Q2 are 2N3904 (standard EBC pinout); U27 is a DS1233-5 CPU
supervisor, electrically unrelated but also a genuine 3-pin TO-92
package (GND/RESET/VCC). Verified both real pinouts already match the
existing pad-to-net mapping (pad1/2/3 = E/B/C for the 2N3904s,
GND/RESET/VCC for the DS1233) - footprint pad numbers are position
slots, not semantics, so this carries no pin-swap risk.

All three share identical 2.54mm inline pad spacing; official
Package_TO_SOT_THT:TO-92_Inline_Wide is an exact match ("TO-92 leads
in-line, wide", NXP SOT54/SC-43A - precisely this hand-formed
straight-lead mounting style).

Corrected the anchor-point placement shift (old footprint centered on
pad 2, official anchors at pad 1) immediately this time rather than
after the fact - verified via DRC that no track_dangling/starved_thermal
regressions appeared, unlike the first pass on R/C/D.

Co-Authored-By: Claude Sonnet 5 <noreply@anthropic.com>
Parts:
- Q2: footprint My_Components:Transistor_TO92_EBC_254 -> Package_TO_SOT_THT:TO-92_Inline_Wide
Changed lines of the file:
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@@
 			)
 		)
-		(property "Footprint" "My_Components:Transistor_TO92_EBC_254"
+		(property "Footprint" "Package_TO_SOT_THT:TO-92_Inline_Wide"
 			(at 175.26 152.4 0)
 			(hide yes)

Commit message: Relink J5 (D-sub DE9M serial connector) to the official footprint
My_Components:Conn_Dsub_DE9M had a well-matched official candidate
(Connector_Dsub:DSUB-9_Pins_Horizontal_P2.77x2.84mm_EdgePinOffset7.70mm_Housed_MountingHolesOffset9.12mm)
verified pad-for-pad against the board's real geometry: pin pitch,
row spacing, and mounting-hole span all matched within rounding
(2.77/2.84mm generic vs. the exact 2.7432/2.8448mm = 0.108in/0.112in
real dimensions), including the shield/mounting pads sitting at the
vertical center between the two pin rows - ruled out a same-named
"4.94mm" variant that instead places its shield pads at the row-2
height, a genuine mechanical mismatch, not just a naming difference.

The only obstacle to using the official footprint unmodified was a
pad-name mismatch: the schematic symbol's shield pin was numbered
"0", but the official footprint's two shield pads are named "SH".
Rather than fork the footprint into a project-local copy just to
rename two pads (as done for J4), renamed the symbol's pin number
from "0" to "SH" instead - verified this symbol is embedded in only
one schematic file and used by only this one component, and the pin
rename is a pure label change (name stays "GND", no wires move), so
the blast radius is contained to J5 with no other changes required.

Corrected the anchor-point/rotation after forward-annotation: moved
to (202.3364, 17.2974) and rotated 180 degrees. All 11 pads land
within ~0.1mm of their pre-swap positions with unchanged net
assignments (including both SH pads correctly on GND). 3D model
orientation verified visually.

Co-Authored-By: Claude Sonnet 5 <noreply@anthropic.com>
Parts:
- J5: footprint My_Components:Conn_Dsub_DE9M -> Connector_Dsub:DSUB-9_Pins_Horizontal_P2.77x2.84mm_EdgePinOffset7.70mm_Housed_MountingHolesOffset9.12mm
Connections:
- net GND: now also J5.SH (GND); no longer J5.0 (GND)
Changed lines of the file:
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@@
 			)
 		)
-		(property "Footprint" "My_Components:Conn_Dsub_DE9M"
+		(property "Footprint" "Connector_Dsub:DSUB-9_Pins_Horizontal_P2.77x2.84mm_EdgePinOffset7.70mm_Housed_MountingHolesOffset9.12mm"
 			(at 264.16 35.56 0)
 			(hide yes)

Commit message: Relink J6 (13x2 shrouded IDC header) to the official footprint
My_Components:Conn_Pin_Header_13x2_2.54mm_Shrouded (3M/Mouser
517-30326-6002 parallel port header) had a well-matched official
candidate: Connector_IDC:IDC-Header_2x13_P2.54mm_Vertical. Schematic
symbol is the standard Connector_Generic:Conn_02x13_Odd_Even (plain
pin numbers 1-26), so no pad-naming fork was needed - straight
relink.

As flagged in the migration plan, this footprint has the same
axis-arrangement gotcha seen on JP1/JP2 and J6 was called out
specifically: it arranges its 13 columns along local Y (with the
2-pin row-pair along local X), while the board's real layout runs
columns along X. Derived and verified the correction pad-by-pad
across all 26 pins before applying: rotation 270 degrees (not a
simple 180 flip), anchored at pad 1's original world position.

Corrected the anchor-point/rotation after forward-annotation: moved
to (163.83, 11.43) and rotated 270 degrees. All 26 pads land exactly
on their pre-swap world positions with unchanged net assignments. 3D
model orientation verified visually.

Co-Authored-By: Claude Sonnet 5 <noreply@anthropic.com>
Parts:
- J6: footprint My_Components:Conn_Pin_Header_13x2_2.54mm_Shrouded -> Connector_IDC:IDC-Header_2x13_P2.54mm_Vertical
Changed lines of the file:
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@@
 			)
 		)
-		(property "Footprint" "My_Components:Conn_Pin_Header_13x2_2.54mm_Shrouded"
+		(property "Footprint" "Connector_IDC:IDC-Header_2x13_P2.54mm_Vertical"
 			(at 116.84 134.62 0)
 			(hide yes)
