File: KiCad/Radio-86RK-IO.kicad_sch (KiCad schematic)
At the start: 16 parts, among them J5 Serial, J6 Parallel, Q2 2N3904, U16 7486/К155ЛП5, U20 7400/К155ЛА3, U22 SN75154N/К170УП2В, U23 SN75150P/К170АП2, U24 SN75150P/К170АП2, U3 8251A/КР580ВВ51А, U4 8253/КР580ВИ53, U6 8255A/КР580ВВ55А

Commit message: Relink SP1 (12mm speaker) to a materialized custom footprint
Real part is PUI Audio AT-1224-TWT-R (Mouser 665-AT-1224TWTR), a
12mm magnetic transducer. No official KiCad footprint exists for
this part. Sourced the manufacturer's own KiCad library export
(SamacSys/Ultra Librarian) with the exact real part number,
converted its legacy footprint format to modern KiCad 10 syntax,
and verified it against the manufacturer datasheet mechanical
drawing (Ø12mm body, 6.5mm pin pitch, 2x0.6mm pin holes - all
matching pad-for-pad). Includes the manufacturer's real STEP 3D
model.

New footprint anchors at pad1 (local origin) with pads running
along local +Y, versus the project's center-anchored, 180°-rotated
instance. Solved for the correction via the established rotation
transform (position (254.559, 13.97) = old pad1 world location,
90° rotation) and verified both pads land within 0.002mm of their
pre-swap world positions, nets unchanged (Net-(R1-Pad2), VCC).

DRC lib_footprint_issues 26 -> 25.
Parts:
- SP1: footprint My_Components:Speaker_12mm -> Speaker_Custom:AT-1224-TWT-R
Changed lines of the file:
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@@
 			)
 		)
-		(property "Footprint" "My_Components:Speaker_12mm"
+		(property "Footprint" "Speaker_Custom:AT-1224-TWT-R"
 			(at 180.34 134.62 0)
 			(hide yes)
