File: KiCad/Radio-86RK-IO.kicad_sch (KiCad schematic)
At the start: 16 parts, among them J5 Serial, J6 Parallel, Q2 2N3904, U16 7486/К155ЛП5, U20 7400/К155ЛА3, U22 SN75154N/К170УП2В, U23 SN75150P/К170АП2, U24 SN75150P/К170АП2, U3 8251A/КР580ВВ51А, U4 8253/КР580ВИ53, U6 8255A/КР580ВВ55А

Commit message: Relink U21/U23/U24 (8-pin DIP ICs) to a materialized socket+chip composite footprint
Package width confirmed 300mil DIP-8 against TL071 (TI: "P (PDIP, 8)") and
SN75150P (TI: "P PDIP 8", 13.97mm tube width) datasheets, matching the
board's existing 7.62mm row spacing.

New IC_Socket_Custom:DIP-8_W7.62mm_Socketed footprint reuses the official
Package_DIP:DIP-8_W7.62mm_Socket pads/silkscreen, with two composited 3D
models: the official socket STEP at board level plus the official bare-chip
STEP raised 5.1mm in Z (real stack height of the BOM socket, Mouser
649-DILB8P223TLF) so the chip renders seated in its socket. Both models are
official KiCad Package_DIP assets - no missing-model gap this time.

Anchor point moved from array-center (old hand-drawn footprint) to pad1
(official footprint convention); required rotation recomputed from scratch
per-instance (90 -> 180) rather than trusting F8's preserved old rotation
value, verified against all 8 pads/nets per instance before committing.

Co-Authored-By: Claude Sonnet 5 <noreply@anthropic.com>
Parts:
- U23, U24: footprint My_Components:IC_DIP8_300 -> IC_Socket_Custom:DIP-8_W7.62mm_Socketed
Changed lines of the file:
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@@
 			)
 		)
-		(property "Footprint" "My_Components:IC_DIP8_300"
+		(property "Footprint" "IC_Socket_Custom:DIP-8_W7.62mm_Socketed"
 			(at 208.28 45.72 0)
 			(hide yes)
@@
 			)
 		)
-		(property "Footprint" "My_Components:IC_DIP8_300"
+		(property "Footprint" "IC_Socket_Custom:DIP-8_W7.62mm_Socketed"
 			(at 208.28 83.82 0)
 			(hide yes)

Commit message: Relink U15-U20 (14-pin DIP 74LS-series logic) to the socket+chip composite footprint
Package width confirmed 300mil DIP-14 for the 74LS family (SN74LS00N: TI "N
package" PDIP-14), matching the board's existing 7.62mm row spacing. Reuses
the Task 23 IC_Socket_Custom compositing approach: pads/silkscreen from the
official Package_DIP:DIP-14_W7.62mm_Socket footprint, plus two composited
3D models (official socket STEP at board level, official chip STEP raised
5.48mm - real stack height of the BOM socket, Mouser 649-DILB14P-223TLF).

All 6 references are multi-unit symbols with redundant per-unit Footprint
property copies spread across up to 4 sheet files each (26 unit-instance
copies total) - batch_edit_schematic_components only patches one instance
per reference per call, so remaining stragglers were located and verified
by reference before a direct text substitution.

Anchor point moved from array-center to pad1 and rotation recomputed
180 (from F8's preserved 90) per instance, verified: all six show the
correct universal 74-series DIP-14 power pinout (pad7=GND, pad14=VCC),
and U15's full pad/net list matches the pre-swap board exactly.

Co-Authored-By: Claude Sonnet 5 <noreply@anthropic.com>
Parts:
- U16, U20: footprint My_Components:IC_DIP14_300 -> IC_Socket_Custom:DIP-14_W7.62mm_Socketed
Changed lines of the file:
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@@
 			)
 		)
-		(property "Footprint" "My_Components:IC_DIP14_300"
+		(property "Footprint" "IC_Socket_Custom:DIP-14_W7.62mm_Socketed"
 			(at 149.86 99.06 0)
 			(hide yes)
@@
 			)
 		)
-		(property "Footprint" "My_Components:IC_DIP14_300"
+		(property "Footprint" "IC_Socket_Custom:DIP-14_W7.62mm_Socketed"
 			(at 129.54 86.36 0)
 			(hide yes)
@@
 			)
 		)
-		(property "Footprint" "My_Components:IC_DIP14_300"
+		(property "Footprint" "IC_Socket_Custom:DIP-14_W7.62mm_Socketed"
 			(at 129.54 101.6 0)
 			(hide yes)
