File: KiCad/Radio-86RK-IO.kicad_sch (KiCad schematic)
At the start: 16 parts, among them J5 Serial, J6 Parallel, Q2 2N3904, U16 7486/К155ЛП5, U20 7400/К155ЛА3, U22 SN75154N/К170УП2В, U23 SN75150P/К170АП2, U24 SN75150P/К170АП2, U3 8251A/КР580ВВ51А, U4 8253/КР580ВИ53, U6 8255A/КР580ВВ55А

Commit message: Relink U2/U14/U22 (16-pin DIP ICs) to the socket+chip composite footprint
Package width confirmed 300mil DIP-16 against the Intel 8224 datasheet
("16-Lead Cerdip Package") and TI SN75154N datasheet ("N PDIP 16", 13.97mm
tube width - the same standard TI 300mil tube spec confirmed for SN75150P
in Task 23); 74LS138 already covered by the Task 24 74LS-family confirmation.
Matches the board's existing 7.62mm row spacing.

Reuses the Task 23 IC_Socket_Custom compositing approach: pads/silkscreen
from the official Package_DIP:DIP-16_W7.62mm_Socket footprint, plus two
composited 3D models (official socket STEP at board level, official chip
STEP raised 5.48mm - real stack height of the BOM socket, Mouser
649-DILB16P-223TLF, per Arrow/Mouser structured spec data).

All three are single-unit symbols with one placement each - no multi-unit
stragglers this time. Anchor point moved from array-center to pad1 and
rotation recomputed 180 (from F8's preserved 90) per instance; U2's full
pad/net list matches the pre-swap board exactly, and U14/U22 both show
correct standard pinouts (74LS138 pin8=GND/pin16=VCC; SN75154N pin8=GND).

Co-Authored-By: Claude Sonnet 5 <noreply@anthropic.com>
Parts:
- U22: footprint My_Components:IC_DIP16_300 -> IC_Socket_Custom:DIP-16_W7.62mm_Socketed
Changed lines of the file:
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@@
 			)
 		)
-		(property "Footprint" "My_Components:IC_DIP16_300"
+		(property "Footprint" "IC_Socket_Custom:DIP-16_W7.62mm_Socketed"
 			(at 208.28 147.32 0)
 			(hide yes)

Commit message: Relink U4/U13 (24-pin DIP ICs) to the socket+chip composite footprint
Package width confirmed 600mil DIP-24 - the board's own measured 15.24mm row
spacing already matched Package_DIP:DIP-24_W15.24mm exactly, and both real
parts (Intel 8253 PIT, TI SN74198N shift register) are standard 24-pin
plastic DIPs, a package size with no narrow-body variant in common use
(unlike the 20-pin case in Task 26 where both widths genuinely exist).

Reuses the Task 23 IC_Socket_Custom compositing approach: pads/silkscreen
from the official Package_DIP:DIP-24_W15.24mm_Socket footprint, plus two
composited 3D models (official socket STEP at board level, official chip
STEP raised 5.48mm). Stack height carried over from the same Amphenol TLF-
family figure confirmed for the 14/16-pin sockets, cross-checked against a
directly-found 24-pin sibling part (DILB24P-224TLF) which also lists 5.48mm.

Anchor point moved from array-center to pad1 and rotation recomputed 180
(from F8's preserved 90) per instance; U4's full pad/net list matches the
pre-swap board exactly, and U13 shows the correct standard 24-pin pinout
(pin12=GND, pin24=VCC).

Co-Authored-By: Claude Sonnet 5 <noreply@anthropic.com>
Parts:
- U4: footprint My_Components:IC_DIP24_600 -> IC_Socket_Custom:DIP-24_W15.24mm_Socketed
Changed lines of the file:
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@@
 			)
 		)
-		(property "Footprint" "My_Components:IC_DIP24_600"
+		(property "Footprint" "IC_Socket_Custom:DIP-24_W15.24mm_Socketed"
 			(at 71.12 48.26 0)
 			(hide yes)

Commit message: Relink U3/U9/U10/U11 (28-pin DIP ICs) to the socket+chip composite footprint
Package width confirmed 600mil DIP-28 - the board's own measured 15.24mm row
spacing already matched Package_DIP:DIP-28_W15.24mm exactly, and the
Alliance Memory AS6C62256 datasheet explicitly specifies "28 pin 600 mil
PDIP"; the Intel 8251A and 2764/28C64-family EPROM parts are standard
28-pin plastic DIPs with no narrow-body variant in common use for this era.

Reuses the Task 23 IC_Socket_Custom compositing approach: pads/silkscreen
from the official Package_DIP:DIP-28_W15.24mm_Socket footprint, plus two
composited 3D models (official socket STEP at board level, official chip
STEP raised 5.48mm - stack height directly confirmed this time for the BOM
socket, Mouser 649-DILB28P223TLF).

Anchor point moved from array-center to pad1 and rotation recomputed 180
(from F8's preserved 90) per instance; U3's full pad/net list matches the
pre-swap board exactly, and U9/U10/U11 all show the correct standard 28-pin
memory pinout (pin14=GND, pin28=VCC).

Co-Authored-By: Claude Sonnet 5 <noreply@anthropic.com>
Parts:
- U3: footprint My_Components:IC_DIP28_600 -> IC_Socket_Custom:DIP-28_W15.24mm_Socketed
Changed lines of the file:
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@@
 			)
 		)
-		(property "Footprint" "My_Components:IC_DIP28_600"
+		(property "Footprint" "IC_Socket_Custom:DIP-28_W15.24mm_Socketed"
 			(at 142.24 52.07 0)
 			(hide yes)

Commit message: Relink U1/U5/U6/U7/U8 (40-pin DIP ICs) to the socket+chip composite footprint
Package width confirmed 600mil DIP-40 - the board's own measured 15.24mm row
spacing already matched Package_DIP:DIP-40_W15.24mm exactly, and the Intel
8080A/8255A/8257/8275 family is universally packaged in standard 40-pin
plastic DIP with no narrow-body variant.

Reuses the Task 23 IC_Socket_Custom compositing approach: pads/silkscreen
from the official Package_DIP:DIP-40_W15.24mm_Socket footprint, plus two
composited 3D models (official socket STEP at board level, official chip
STEP raised 5.48mm - stack height directly confirmed for the BOM socket,
Mouser 649-DILB40P223TLF).

Anchor point moved from array-center to pad1 and rotation recomputed 180
(from F8's preserved 90) per instance; U1's full pad/net list matches the
pre-swap board exactly, and U5/U6/U7/U8 all show correct standard 40-pin
pinouts (GND/VCC at the expected positions).

This is the last unresolved My_Components reference in the project - DRC
confirms the "lib_footprint_issues" category has dropped to 0 (from 21
after Task 23), matching the plan's expected end state for the IC tasks.

Co-Authored-By: Claude Sonnet 5 <noreply@anthropic.com>
Parts:
- U6: footprint My_Components:IC_DIP40_600 -> IC_Socket_Custom:DIP-40_W15.24mm_Socketed
Changed lines of the file:
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@@
 			)
 		)
-		(property "Footprint" "My_Components:IC_DIP40_600"
+		(property "Footprint" "IC_Socket_Custom:DIP-40_W15.24mm_Socketed"
 			(at 71.12 151.13 0)
 			(hide yes)
