File: KiCad/Radio-86RK-IO.kicad_sch (KiCad schematic)
At the start: 16 parts, among them J5 Serial, J6 Parallel, Q2 2N3904, U16 7486/К155ЛП5, U20 7400/К155ЛА3, U22 SN75154N/К170УП2В, U23 SN75150P/К170АП2, U24 SN75150P/К170АП2, U3 8251A/КР580ВВ51А, U4 8253/КР580ВИ53, U6 8255A/КР580ВВ55А

Commit message: Re-home 8255A (PPI) from lost my_components library
Step 12/18. Relinks U5 on the Keyboard sheet and U6 on the IO sheet from
my_components:8255A to Radio86RK_Custom:8255A (same part used on both
sheets).
Parts:
- U6: symbol my_components:8255A -> Radio86RK_Custom:8255A
Changed lines of the file:
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@@
 	)
 	(symbol
-		(lib_id "my_components:8255A")
+		(lib_id "Radio86RK_Custom:8255A")
 		(at 71.12 151.13 0)
 		(unit 1)

Commit message: Re-home 8251A (USART) from lost my_components library
Step 13/18. Relinks U3 on the IO sheet from my_components:8251A to
Radio86RK_Custom:8251A.
Parts:
- U3: symbol my_components:8251A -> Radio86RK_Custom:8251A
Changed lines of the file:
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@@
 	)
 	(symbol
-		(lib_id "my_components:8251A")
+		(lib_id "Radio86RK_Custom:8251A")
 		(at 142.24 52.07 0)
 		(unit 1)

Commit message: Re-home 8254 (PIT) from lost my_components library
Step 14/18. Relinks U4 on the IO sheet from my_components:8254 to
Radio86RK_Custom:8254.
Parts:
- U4: symbol my_components:8254 -> Radio86RK_Custom:8254
Changed lines of the file:
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@@
 	)
 	(symbol
-		(lib_id "my_components:8254")
+		(lib_id "Radio86RK_Custom:8254")
 		(at 71.12 48.26 0)
 		(unit 1)

Commit message: Re-home SN75150P (RS-232 line driver) from lost my_components library
Step 15/18. Relinks U23 and U24 on the IO sheet from my_components:SN75150P
to Radio86RK_Custom:SN75150P.
Parts:
- U23, U24: symbol my_components:SN75150P -> Radio86RK_Custom:SN75150P
Changed lines of the file:
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@@
 	)
 	(symbol
-		(lib_id "my_components:SN75150P")
+		(lib_id "Radio86RK_Custom:SN75150P")
 		(at 208.28 34.29 0)
 		(unit 1)
@@
 	)
 	(symbol
-		(lib_id "my_components:SN75150P")
+		(lib_id "Radio86RK_Custom:SN75150P")
 		(at 208.28 72.39 0)
 		(unit 1)

Commit message: Re-home DE9 (RS-232 D-sub connector) from lost my_components library
Step 16/18. Relinks J5 on the IO sheet from my_components:DE9 to
Radio86RK_Custom:DE9.
Parts:
- J5: symbol my_components:DE9 -> Radio86RK_Custom:DE9
Changed lines of the file:
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@@
 	)
 	(symbol
-		(lib_id "my_components:DE9")
+		(lib_id "Radio86RK_Custom:DE9")
 		(at 261.62 35.56 0)
 		(unit 1)

Commit message: Re-home SN75154P (RS-232 line receiver) from lost my_components library
Step 18/18 (final). Relinks U22 on the IO sheet from
my_components:SN75154P to Radio86RK_Custom:SN75154P.

Unlike the original monolithic relink (28c05ca on migrate2kicad10), this
text-level lib_id swap never touches the instance's (at ...)/(mirror y)
placement transform, so U22's mirror is preserved automatically. This is
the root-cause fix for the U3/U22 ERC errors previously misdiagnosed and
filed as GitHub issue #2 ("pre-existing RS-232 wiring defect") -- the real
cause was 28c05ca silently dropping this mirror, which reassigns which
physical pin each fixed wire coordinate connects to without touching a
single wire.

All 18 parts now re-homed from the lost my_components library into the
project-local Radio86RK_Custom.kicad_sym, one part per commit.

ERC: 32 violations / 0 errors (down from 52/0 after step 1; the 13
U3/U22 pin_not_driven/pin_not_connected errors that 28c05ca introduced
never appeared in this replay). Remaining 32 violations are all
same_local_global_label warnings, unrelated to this fix.
Parts:
- U22: symbol my_components:SN75154P -> Radio86RK_Custom:SN75154P
Changed lines of the file:
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@@
 	)
 	(symbol
-		(lib_id "my_components:SN75154P")
+		(lib_id "Radio86RK_Custom:SN75154P")
 		(at 208.28 123.19 0)
 		(mirror y)
