File: KiCad/Radio-86RK-CRT-Mem.kicad_sch (KiCad schematic)
At the start: 22 parts, among them J1 Video, Q1 2N3904, U10 2764/К573РФ6/28C64, U11 2764/К573РФ6/28C64, U13 74198/К155ИР13, U15 7492/К155ИЕ4, U16 7486/К155ЛП5, U17 7474/К155ТМ2, U18 7408/К155ЛИ1, U19 7404/К155ЛН1, U8 8275/КР580ВГ75, U9 AS6C62256

Commit message: Relink R1-R15 to official Resistor_THT footprint
The 15 discrete resistors used My_Components:Res_762, an unresolved
library nickname with no fp-lib-table entry anywhere on disk. Compared
the footprint against the actual ordered part (Stackpole CF14 1/4W
carbon film, per the README Mouser BOM) rather than just the closest
official name: the real part's datasheet body (6.50x2.30mm) is closer
to Resistor_THT:R_Axial_DIN0207_L6.3mm_D2.5mm_P7.62mm_Horizontal's
silkscreen outline (6.54x2.74mm) than to the project's own hand-drawn
one (5.84x2.03mm), so the official footprint is the more accurate
choice, not just a fallback. Same 7.62mm pin pitch, and it comes with
a working 3D model - the project's own model reference
("discret/resistor.wrl") doesn't resolve on any current KiCad install.

Co-Authored-By: Claude Sonnet 5 <noreply@anthropic.com>
Parts:
- R10, R2, R3, R5, R9: footprint My_Components:Res_762 -> Resistor_THT:R_Axial_DIN0207_L6.3mm_D2.5mm_P7.62mm_Horizontal
Changed lines of the file:
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@@
 			)
 		)
-		(property "Footprint" "My_Components:Res_762"
+		(property "Footprint" "Resistor_THT:R_Axial_DIN0207_L6.3mm_D2.5mm_P7.62mm_Horizontal"
 			(at 227.33 132.842 90)
 			(hide yes)
@@
 			)
 		)
-		(property "Footprint" "My_Components:Res_762"
+		(property "Footprint" "Resistor_THT:R_Axial_DIN0207_L6.3mm_D2.5mm_P7.62mm_Horizontal"
 			(at 227.33 145.542 90)
 			(hide yes)
@@
 			)
 		)
-		(property "Footprint" "My_Components:Res_762"
+		(property "Footprint" "Resistor_THT:R_Axial_DIN0207_L6.3mm_D2.5mm_P7.62mm_Horizontal"
 			(at 231.902 120.65 90)
 			(hide yes)
@@
 			)
 		)
-		(property "Footprint" "My_Components:Res_762"
+		(property "Footprint" "Resistor_THT:R_Axial_DIN0207_L6.3mm_D2.5mm_P7.62mm_Horizontal"
 			(at 242.062 138.43 90)
 			(hide yes)
@@
 			)
 		)
-		(property "Footprint" "My_Components:Res_762"
+		(property "Footprint" "Resistor_THT:R_Axial_DIN0207_L6.3mm_D2.5mm_P7.62mm_Horizontal"
 			(at 242.062 156.21 90)
 			(hide yes)

Commit message: Relink ceramic capacitors and F1 polyfuse to official footprints
The 39 refs (C1-C32, C39-C44, F1) used My_Components:Cap_Cer_508, an
unresolved library nickname. Resolved the real ordered parts from the
README Mouser BOM: C1-C32 are Vishay K104K15X7RF53H5 (~4.0x4.0x2.6mm
body), C40-C44 are TDK FG28-series (~4.0x5.5mm body), C39 is TDK
FG24-series (~4.5x5.5mm, larger), and F1 is a Littelfuse 16R110BU PTC
resettable fuse with no dedicated KiCad footprint.

All share the project's existing 5.08mm pitch (matches every
datasheet's 5.0mm +/-0.8-1.0mm spec). Split into two official
Capacitor_THT footprints matching the two real body-size groups
(C_Disc_D4.7mm_W2.5mm_P5.00mm for the smaller Vishay/FG28 parts,
C_Disc_D5.1mm_W3.2mm_P5.00mm for the larger FG24 C39) rather than
forcing one footprint on parts of two different real sizes. F1 reuses
the small-cap disc footprint since Littelfuse's radial PTC package at
this pitch is mechanically a disc shape with no official equivalent.

Co-Authored-By: Claude Sonnet 5 <noreply@anthropic.com>
Parts:
- C40: footprint My_Components:Cap_Cer_508 -> Capacitor_THT:C_Disc_D4.7mm_W2.5mm_P5.00mm
Changed lines of the file:
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@@
 			)
 		)
-		(property "Footprint" "My_Components:Cap_Cer_508"
+		(property "Footprint" "Capacitor_THT:C_Disc_D4.7mm_W2.5mm_P5.00mm"
 			(at 254 143.8148 0)
 			(hide yes)

Commit message: Relink electrolytic capacitors C33-C38 to official footprint
The real ordered part is KEMET A750EK476M1E (47uF/25V Radial Solid
Polymer Aluminum, case code EK: D6.3mm x L8mm, 2.5mm lead spacing) -
the project's existing pitch and footprint name already matched this
part exactly, so this is a clean swap: Capacitor_THT:CP_Radial_D6.3mm_P2.50mm
is an essentially exact match (same pitch, near-identical pad/drill,
same pad-numbering/polarity convention) and adds a working 3D model.

Co-Authored-By: Claude Sonnet 5 <noreply@anthropic.com>
Parts:
- C38: footprint My_Components:Cap_Elec_Radial_6.3mm -> Capacitor_THT:CP_Radial_D6.3mm_P2.50mm
Changed lines of the file:
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@@
 			)
 		)
-		(property "Footprint" "My_Components:Cap_Elec_Radial_6.3mm"
+		(property "Footprint" "Capacitor_THT:CP_Radial_D6.3mm_P2.50mm"
 			(at 250.19 149.86 0)
 			(hide yes)

Commit message: Relink transistors Q1/Q2 and U27 to official TO-92 footprint
Q1/Q2 are 2N3904 (standard EBC pinout); U27 is a DS1233-5 CPU
supervisor, electrically unrelated but also a genuine 3-pin TO-92
package (GND/RESET/VCC). Verified both real pinouts already match the
existing pad-to-net mapping (pad1/2/3 = E/B/C for the 2N3904s,
GND/RESET/VCC for the DS1233) - footprint pad numbers are position
slots, not semantics, so this carries no pin-swap risk.

All three share identical 2.54mm inline pad spacing; official
Package_TO_SOT_THT:TO-92_Inline_Wide is an exact match ("TO-92 leads
in-line, wide", NXP SOT54/SC-43A - precisely this hand-formed
straight-lead mounting style).

Corrected the anchor-point placement shift (old footprint centered on
pad 2, official anchors at pad 1) immediately this time rather than
after the fact - verified via DRC that no track_dangling/starved_thermal
regressions appeared, unlike the first pass on R/C/D.

Co-Authored-By: Claude Sonnet 5 <noreply@anthropic.com>
Parts:
- Q1: footprint My_Components:Transistor_TO92_EBC_254 -> Package_TO_SOT_THT:TO-92_Inline_Wide
Changed lines of the file:
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@@
 			)
 		)
-		(property "Footprint" "My_Components:Transistor_TO92_EBC_254"
+		(property "Footprint" "Package_TO_SOT_THT:TO-92_Inline_Wide"
 			(at 246.38 124.46 0)
 			(hide yes)

Commit message: Relink RN1 (10k SIP10 resistor array) to official footprint
Real part is Bourns 4610X-1LF-10K, "bussed" SIP10 topology (1 common
pin + 9 resistors), 2.54mm pitch - matches RN1's existing wiring
exactly (pad 1 = VCC common bus, pads 2-10 = individual pulled-up
signal legs). Resistor_THT:R_Array_SIP10 is an exact match: same
pitch, pad 1 = rect = common-pin convention.

Corrected the anchor-point placement shift immediately (old footprint
centered between pad 1 and pad 10, official anchors at pad 1); all 10
pad positions and net mappings verified identical to pre-swap.

Co-Authored-By: Claude Sonnet 5 <noreply@anthropic.com>
Parts:
- RN1: footprint My_Components:Conn_SIL10 -> Resistor_THT:R_Array_SIP10
Changed lines of the file:
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@@
 			)
 		)
-		(property "Footprint" "My_Components:Conn_SIL10"
+		(property "Footprint" "Resistor_THT:R_Array_SIP10"
 			(at 233.045 25.4 90)
 			(hide yes)

Commit message: Relink JP1/JP2 (4-pin 2.54mm headers) to official footprint
Real part is Amphenol/FCI 68000-204HLF (BOM lists it as TE
Connectivity - minor misattribution, correct manufacturer is
Amphenol/FCI, doesn't affect footprint choice), 4-position 2.54mm
1-row unshrouded header - exact match to
Connector_PinHeader_2.54mm:PinHeader_1x04_P2.54mm_Vertical.

This one had a new wrinkle: unlike every footprint swapped so far,
this official footprint arranges pads along local Y (pad2 at (0,2.54))
rather than local X. The usual rotation carried over from the old
footprint (90) rotated the vertical arrangement into horizontal;
recomputed and corrected to 180, verified all 4 pads on both JP1 and
JP2 match pre-swap positions exactly.

Co-Authored-By: Claude Sonnet 5 <noreply@anthropic.com>
Parts:
- JP1, JP2: footprint My_Components:Conn_Pin_Header_4x1_2.54mm -> Connector_PinHeader_2.54mm:PinHeader_1x04_P2.54mm_Vertical
Changed lines of the file:
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@@
 			)
 		)
-		(property "Footprint" "My_Components:Conn_Pin_Header_4x1_2.54mm"
+		(property "Footprint" "Connector_PinHeader_2.54mm:PinHeader_1x04_P2.54mm_Vertical"
 			(at 20.32 157.48 0)
 			(hide yes)
@@
 			)
 		)
-		(property "Footprint" "My_Components:Conn_Pin_Header_4x1_2.54mm"
+		(property "Footprint" "Connector_PinHeader_2.54mm:PinHeader_1x04_P2.54mm_Vertical"
 			(at 162.56 114.3 0)
 			(hide yes)

Commit message: Relink J1 (RCA phono jack) to a materialized custom footprint
No RCA jack footprint exists in any official or already-installed
third-party KiCad library (searched all 211 entries in Connector_Audio
plus the installed alternate-kicad-library package - zero matches).

Downloaded the manufacturer-verified SnapEDA footprint for the real
part (Same Sky/CUI RCJ-014, Mouser 490-RCJ-014) and compared it
against both the project's existing geometry and the official Same
Sky RCJ-01 series datasheet: the downloaded file's drill sizes
(1.70mm signal / 2.60mm x3 ground) and pad spacing (10.00mm
ground-to-ground, 4.50mm signal-to-odd-ground) match the datasheet
exactly, while the project's own hand-drawn footprint was off by
0.58mm on the signal-to-odd-ground dimension - same pattern as the
earlier resistor finding, the project's own geometry isn't always the
ground truth.

Rebuilt it as a clean modern-format project-local footprint
(Conn_RCA_Custom.pretty/RCJ-014.kicad_mod), re-origining it so the
"anchor" ground pad coincides with the old footprint's placement -
this meant no PCB position/rotation correction was needed for the
component itself, only the intentional ~0.5mm pad shifts reflecting
the corrected real-world spacing. Also fixed the downloaded file's
incorrect description text (it read "DC POWER JACK" from an unrelated
datasheet - a stale copy-paste error in the community metadata, not a
geometry problem) and renumbered pads to match the existing schematic
(pad 1 = signal, pad 2 = the three ground legs).

Included the manufacturer's STEP 3D model. Its native orientation
didn't match KiCad's placement convention (needed rotation on X/Z, not
just a simple flip) - corrected interactively in the KiCad 3D model
editor and captured the resulting transform (offset 5.5,0,7 / rotate
-90,0,-180) into the library file.

Co-Authored-By: Claude Sonnet 5 <noreply@anthropic.com>
Parts:
- J1: footprint My_Components:Conn_RCA_Right -> Conn_RCA_Custom:RCJ-014
Changed lines of the file:
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@@
 			)
 		)
-		(property "Footprint" "My_Components:Conn_RCA_Right"
+		(property "Footprint" "Conn_RCA_Custom:RCJ-014"
 			(at 264.16 149.86 0)
 			(hide yes)

Commit message: Relink U15-U20 (14-pin DIP 74LS-series logic) to the socket+chip composite footprint
Package width confirmed 300mil DIP-14 for the 74LS family (SN74LS00N: TI "N
package" PDIP-14), matching the board's existing 7.62mm row spacing. Reuses
the Task 23 IC_Socket_Custom compositing approach: pads/silkscreen from the
official Package_DIP:DIP-14_W7.62mm_Socket footprint, plus two composited
3D models (official socket STEP at board level, official chip STEP raised
5.48mm - real stack height of the BOM socket, Mouser 649-DILB14P-223TLF).

All 6 references are multi-unit symbols with redundant per-unit Footprint
property copies spread across up to 4 sheet files each (26 unit-instance
copies total) - batch_edit_schematic_components only patches one instance
per reference per call, so remaining stragglers were located and verified
by reference before a direct text substitution.

Anchor point moved from array-center to pad1 and rotation recomputed
180 (from F8's preserved 90) per instance, verified: all six show the
correct universal 74-series DIP-14 power pinout (pad7=GND, pad14=VCC),
and U15's full pad/net list matches the pre-swap board exactly.

Co-Authored-By: Claude Sonnet 5 <noreply@anthropic.com>
Parts:
- U15, U16, U17, U18, U19: footprint My_Components:IC_DIP14_300 -> IC_Socket_Custom:DIP-14_W7.62mm_Socketed
Changed lines of the file:
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@@
 			)
 		)
-		(property "Footprint" "My_Components:IC_DIP14_300"
+		(property "Footprint" "IC_Socket_Custom:DIP-14_W7.62mm_Socketed"
 			(at 213.36 134.62 0)
 			(hide yes)
@@
 			)
 		)
-		(property "Footprint" "My_Components:IC_DIP14_300"
+		(property "Footprint" "IC_Socket_Custom:DIP-14_W7.62mm_Socketed"
 			(at 175.26 124.46 0)
 			(hide yes)
@@
 			)
 		)
-		(property "Footprint" "My_Components:IC_DIP14_300"
+		(property "Footprint" "IC_Socket_Custom:DIP-14_W7.62mm_Socketed"
 			(at 213.36 121.92 0)
 			(hide yes)
@@
 			)
 		)
-		(property "Footprint" "My_Components:IC_DIP14_300"
+		(property "Footprint" "IC_Socket_Custom:DIP-14_W7.62mm_Socketed"
 			(at 213.36 147.32 0)
 			(hide yes)
@@
 			)
 		)
-		(property "Footprint" "My_Components:IC_DIP14_300"
+		(property "Footprint" "IC_Socket_Custom:DIP-14_W7.62mm_Socketed"
 			(at 124.46 157.48 0)
 			(hide yes)
@@
 			)
 		)
-		(property "Footprint" "My_Components:IC_DIP14_300"
+		(property "Footprint" "IC_Socket_Custom:DIP-14_W7.62mm_Socketed"
 			(at 152.4 160.02 0)
 			(hide yes)
@@
 			)
 		)
-		(property "Footprint" "My_Components:IC_DIP14_300"
+		(property "Footprint" "IC_Socket_Custom:DIP-14_W7.62mm_Socketed"
 			(at 175.26 154.94 0)
 			(hide yes)
