File: KiCad/Radio-86RK-CRT-Mem.kicad_sch (KiCad schematic)
At the start: 22 parts, among them J1 Video, Q1 2N3904, U10 2764/К573РФ6/28C64, U11 2764/К573РФ6/28C64, U13 74198/К155ИР13, U15 7492/К155ИЕ4, U16 7486/К155ЛП5, U17 7474/К155ТМ2, U18 7408/К155ЛИ1, U19 7404/К155ЛН1, U8 8275/КР580ВГ75, U9 AS6C62256

Commit message: Relink Q1/Q2 from stale Device:Q_NPN_EBC to Transistor_BJT:Q_NPN_EBC
The symbol moved libraries between KiCad versions (same name, same E/B/C
pinout) -- Device no longer carries it in KiCad 10. Resolves 2 ERC
lib_symbol_issues warnings. Also includes a mop-up Update Symbol from
Library pass to clear an incidental lib_symbol_mismatch regression the
relink introduced on U19/U20's cached copies in the same files (metadata-
only, Datasheet/Description fields, no connectivity impact).

Co-Authored-By: Claude Sonnet 5 <noreply@anthropic.com>
Parts:
- removed Q1: 2N3904, Package_TO_SOT_THT:TO-92_Inline_Wide, symbol Device:Q_NPN_EBC
- added Q1: 2N3904, Package_TO_SOT_THT:TO-92_Inline_Wide, symbol Transistor_BJT:Q_NPN_EBC
Connections:
- net VCC: now also Q1.3 (C)
- net at R10.2, R5.1, R9.1: now also Q1.2 (B)
- net at R2.1: now also Q1.1 (E)
Changed lines of the file:
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@@
-	)
-	(symbol
-		(lib_id "Device:Q_NPN_EBC")
-		(at 241.3 127 0)
-		(unit 1)
-		(body_style 1)
-		(exclude_from_sim no)
-		(in_bom yes)
-		(on_board yes)
-		(in_pos_files yes)
-		(dnp no)
-		(property "Reference" "Q1"
-			(at 240.03 123.19 0)
-			(show_name no)
-			(do_not_autoplace no)
-			(effects
-				(font
-					(size 1.27 1.27)
-				)
-				(justify right)
-			)
-		)
-		(property "Value" "2N3904"
-			(at 242.57 132.08 0)
-			(show_name no)
-			(do_not_autoplace no)
-			(effects
-				(font
-					(size 1.27 1.27)
-				)
-				(justify right)
-			)
-		)
-		(property "Footprint" "Package_TO_SOT_THT:TO-92_Inline_Wide"
-			(at 246.38 124.46 0)
-			(hide yes)
-			(show_name no)
-			(do_not_autoplace no)
-			(effects
-				(font
-					(size 1.27 1.27)
-				)
-			)
-		)
-		(property "Datasheet" ""
-			(at 241.3 127 0)
-			(show_name no)
-			(do_not_autoplace no)
-			(effects
-				(font
-					(size 1.27 1.27)
-				)
-			)
-		)
-		(property "Description" ""
-			(at 241.3 127 0)
-			(show_name no)
-			(do_not_autoplace no)
-			(effects
-				(font
-					(size 1.27 1.27)
-				)
-			)
-		)
-		(pin "1"
-		)
-		(pin "2"
-		)
-		(pin "3"
-		)
-		(instances
-			(project "Radio-86RK"
-				(path "/8e697b96-cf4c-43ef-b321-8c2422b088bf/00000000-0000-0000-0000-000061d307f8"
-					(reference "Q1")
-					(unit 1)
-				)
-			)
-		)
 	)
 	(symbol
@@
 					(unit 1)
 				)
+			)
+		)
+	)
+	(symbol
+		(lib_id "Transistor_BJT:Q_NPN_EBC")
+		(at 241.3 127 0)
+		(unit 1)
+		(body_style 1)
+		(exclude_from_sim no)
+		(in_bom yes)
+		(on_board yes)
+		(in_pos_files yes)
+		(dnp no)
+		(property "Reference" "Q1"
+			(at 246.38 128.27 0)
+			(show_name no)
+			(do_not_autoplace no)
+			(effects
+				(font
+					(size 1.27 1.27)
+				)
+				(justify left)
+			)
+		)
+		(property "Value" "2N3904"
+			(at 246.38 125.73 0)
+			(show_name no)
+			(do_not_autoplace no)
+			(effects
+				(font
+					(size 1.27 1.27)
+				)
+				(justify left)
+			)
+		)
+		(property "Footprint" "Package_TO_SOT_THT:TO-92_Inline_Wide"
+			(at 246.38 129.54 0)
+			(hide yes)
+			(show_name no)
+			(do_not_autoplace no)
+			(effects
+				(font
+					(size 1.27 1.27)
+				)
+			)
+		)
+		(property "Datasheet" ""
+			(at 241.3 127 0)
+			(hide yes)
+			(show_name no)
+			(do_not_autoplace no)
+			(effects
+				(font
+					(size 1.27 1.27)
+				)
+			)
+		)
+		(property "Description" "NPN transistor, emitter/base/collector"
+			(at 241.3 127 0)
+			(hide yes)
+			(show_name no)
+			(do_not_autoplace no)
+			(effects
+				(font
+					(size 1.27 1.27)
+				)
+			)
+		)
+		(property "Sim.Device" "NPN"
+			(at 241.3 127 0)
+			(hide yes)
+			(show_name no)
+			(do_not_autoplace no)
+			(effects
+				(font
+					(size 1.27 1.27)
+				)
+			)
+		)
+		(property "Sim.Pins" "1=E 2=B 3=C"
+			(at 241.3 127 0)
+			(hide yes)
+			(show_name no)
+			(do_not_autoplace no)
+			(effects
+				(font
+					(size 1.27 1.27)
+				)
+			)
+		)
+		(pin "1"
+		)
+		(pin "2"
+		)
+		(pin "3"
+		)
+		(instances
+			(project "Radio-86RK"
+				(path "/8e697b96-cf4c-43ef-b321-8c2422b088bf/00000000-0000-0000-0000-000061d307f8"
+					(reference "Q1")
+					(unit 1)
+				)
