File: KiCad/Radio-86RK-CRT-Mem.kicad_sch (KiCad schematic)
At the start: 22 parts, among them J1 Video, Q1 2N3904, U10 2764/К573РФ6/28C64, U11 2764/К573РФ6/28C64, U13 74198/К155ИР13, U15 7492/К155ИЕ4, U16 7486/К155ЛП5, U17 7474/К155ТМ2, U18 7408/К155ЛИ1, U19 7404/К155ЛН1, U8 8275/КР580ВГ75, U9 AS6C62256

Commit message: Re-home AS6C62256 (SRAM) from lost my_components library
Step 7/18. Relinks U9 on the CRT-Mem sheet from my_components:AS6C62256 to
Radio86RK_Custom:AS6C62256.
Parts:
- U9: symbol my_components:AS6C62256 -> Radio86RK_Custom:AS6C62256
Changed lines of the file:
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@@
 	)
 	(symbol
-		(lib_id "my_components:AS6C62256")
+		(lib_id "Radio86RK_Custom:AS6C62256")
 		(at 68.58 66.04 0)
 		(unit 1)

Commit message: Re-home 27C64 (EPROM) from lost my_components library
Step 8/18. Relinks U10 and U11 on the CRT-Mem sheet from
my_components:27C64 to Radio86RK_Custom:27C64.
Parts:
- U10, U11: symbol my_components:27C64 -> Radio86RK_Custom:27C64
Changed lines of the file:
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@@
 	)
 	(symbol
-		(lib_id "my_components:27C64")
+		(lib_id "Radio86RK_Custom:27C64")
 		(at 68.58 144.78 0)
 		(unit 1)
@@
 	)
 	(symbol
-		(lib_id "my_components:27C64")
+		(lib_id "Radio86RK_Custom:27C64")
 		(at 190.5 76.2 0)
 		(unit 1)

Commit message: Re-home 74198 (octal D-type flip-flop) from lost my_components library
Step 9/18. Relinks U13 on the CRT-Mem sheet from my_components:74198 to
Radio86RK_Custom:74198.
Parts:
- U13: symbol my_components:74198 -> Radio86RK_Custom:74198
Changed lines of the file:
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@@
 	)
 	(symbol
-		(lib_id "my_components:74198")
+		(lib_id "Radio86RK_Custom:74198")
 		(at 243.84 71.12 0)
 		(unit 1)

Commit message: Re-home 8275 (CRT controller) from lost my_components library
Step 10/18. Relinks U8 on the CRT-Mem sheet from my_components:8275 to
Radio86RK_Custom:8275.
Parts:
- U8: symbol my_components:8275 -> Radio86RK_Custom:8275
Changed lines of the file:
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@@
 	)
 	(symbol
-		(lib_id "my_components:8275")
+		(lib_id "Radio86RK_Custom:8275")
 		(at 127 74.93 0)
 		(unit 1)
